Commit message: (mini_max_defs) add new arm_base_link

File: mini_max/mini_max_defs/urdf/arm.urdf.xacro (robot description, xacro)
@@ -5,9 +5,16 @@
   <property name="arm_major_length" value="0.09208" />
   <macro name="mini_arm" params="name parent *origin">
+    <!-- Arm Base -->
+    <joint name="${name}_base_joint" type="fixed">
+      <insert_block name="origin" />
+      <parent link="${parent}_link"/>
+      <child link="${name}_base_link"/>
+    </joint>
+    <link name="${name}_base_link" />
     <!-- Shoulder pan -->
     <joint name="${name}_shoulder_pan_joint" type="revolute">
       <axis xyz="0 0 1" />
       <insert_block name="origin" />
-      <parent link="${parent}_link"/>
+      <parent link="${name}_base_link"/>
       <child link="${name}_shoulder_pan_link"/>
       <limit lower="-1.57"  upper="1.57" effort="5.0" velocity="5" />

File: mini_max/mini_max_defs/urdf/mini_max.urdf.xacro (robot description, xacro)
@@ -114,6 +114,6 @@
     <origin xyz="0.104775 -0.0381 ${create_height+standoff_height+material_thickness}"/>
   </mini_arm>
-  <!--<mini_gripper name="gripper" parent="arm_wrist_flex">
+  <mini_gripper name="gripper" parent="arm_wrist_flex">
     <origin xyz="0.100 0 0" />
-  </mini_gripper>-->
+  </mini_gripper>
 </robot>

Commit message: (mini_max_defs) drop back to previous port names

File: mini_max/mini_max_defs/urdf/arm.urdf.xacro (robot description, xacro)
@@ -15,5 +15,5 @@
     <joint name="${name}_shoulder_pan_joint" type="revolute">
       <axis xyz="0 0 1" />
-      <insert_block name="origin" />
+      <origin xyz="0 0 0" rpy="0 0 0"/>
       <parent link="${name}_base_link"/>
       <child link="${name}_shoulder_pan_link"/>

Commit message: (mini_max_defs) finalize gripper STL/URDF, add launch file for arm server

File: mini_max/mini_max_defs/urdf/arm.urdf.xacro (robot description, xacro)
@@ -76,8 +76,8 @@
     <link name="${name}_wrist_flex_link">
       <visual name="${name}_wrist_flex_visual">
-        <origin xyz="${0.030/2} 0 0" rpy="0 0 0" />
+        <origin xyz="${0.050/2} 0 0" rpy="0 0 0" />
         <geometry name="${name}_wrist_flex_visual_geom">
           <!--<mesh filename="package://pr2_defs/meshes/wrist_flex.stl" />-->
-          <box size="0.030 0.057 0.040"/>
+          <box size="0.05 0.050 ${ax12_depth}"/>
         </geometry>
         <material name="Orange" />

File: mini_max/mini_max_defs/urdf/gripper.urdf.xacro (robot description, xacro)
@@ -1,34 +1,40 @@
 <?xml version="1.0"?>
 <robot>
-  <macro name="gripper_finger" params="prefix parent reflect">
-    <joint name="${prefix}_finger_joint" type="revolute">
+  <macro name="mini_gripper" params="name parent">
+    <!-- Static Side -->
+    <joint name="${name}_static_joint" type="fixed">
       <axis xyz="0 0 1" />
-      <origin xyz="-0.012 ${reflect*0.033/2} 0" rpy="0 0 0" />
+      <origin xyz="0.1 0 0" rpy="0 0 0" />
+      <parent link="${parent}_link"/>
+      <child link="${name}_link"/>
+    </joint>
+    <link name="${name}_link">
+      <visual name="${name}_static_visual">
+        <origin xyz="-0.05 0.025 0" rpy="-1.57 0 0"/>
+        <geometry name="${name}_static_visual_geom">
+          <mesh filename="package://mini_max_defs/meshes/gripper.stl" />
+        </geometry>
+        <material name="Grey" />
+      </visual>
+      <!-- TODO: add collision -->
+    </link>
+    <!-- Actuated Side -->
+    <joint name="${name}_joint" type="revolute">
+      <axis xyz="0 0 1" />
+      <origin xyz="0.05 -0.025 0" rpy="0 0 0" />
       <limit lower="-1.57"  upper="1.57" effort="5.0" velocity="5" />
       <parent link="${parent}_link"/>
-      <child link="${prefix}_finger_link"/>
+      <child link="finger_link"/>
     </joint>
-    <link name="${prefix}_finger_link">
-      <visual name="${prefix}_finger_visual">
-        <origin xyz="0 0 0" rpy="0 0 0" />
-        <geometry name="${prefix}_finger_visual_geom">
-          <box size="0.125 0.01 0.03"/>
+    <link name="finger_link">
+      <visual name="finger_visual">
+        <origin xyz="0 0 0" rpy="1.57 0 0" />
+        <geometry name="finger_visual_geom">
+          <mesh filename="package://mini_max_defs/meshes/gripper.stl" />
         </geometry>
-        <material name="Orange" />
+        <material name="Grey" />
       </visual>
       <!-- TODO: add collision -->
     </link>
   </macro>
-  <macro name="mini_gripper" params="name parent *origin">
-    <!-- Base of Gripper Pad -->
-    <joint name="${name}_joint" type="fixed">
-      <axis xyz="0 0 1" />
-      <insert_block name="origin" />
-      <parent link="${parent}_link"/>
-      <child link="${name}_link"/>
-    </joint>
-    <link name="${name}_link"/>
-    <gripper_finger prefix="l" parent="gripper" reflect="1"/>
-    <gripper_finger prefix="r" parent="gripper" reflect="-1" />
-  </macro>
 </robot>

File: mini_max/mini_max_defs/urdf/mini_max.urdf.xacro (robot description, xacro)
@@ -114,6 +114,4 @@
     <origin xyz="0.104775 -0.0381 ${create_height+standoff_height+material_thickness}"/>
   </mini_arm>
-  <mini_gripper name="gripper" parent="arm_wrist_flex">
-    <origin xyz="0.100 0 0" />
-  </mini_gripper>
+  <mini_gripper name="gripper" parent="arm_wrist_flex"/>
 </robot>

Commit message: (mini_max_defs) updated URDF

File: mini_max/mini_max_defs/urdf/arm.urdf.xacro (robot description, xacro)
@@ -3,5 +3,6 @@
   <!-- size properties -->
   <property name="arm_pan_height" value="0.00635" />
-  <property name="arm_major_length" value="0.09208" />
+  <!--<property name="arm_major_length" value="0.09208" />-->
+  <property name="arm_major_length" value="0.06627" />
   <macro name="mini_arm" params="name parent *origin">
     <!-- Arm Base -->
@@ -40,7 +41,7 @@
     <link name="${name}_shoulder_lift_link">
       <visual name="${name}_shoulder_lift_visual">
-        <origin xyz="${(ax12_height+arm_major_length)/2} 0 0" rpy="0 0 0" />
+        <origin xyz="${(ax12_center+arm_major_length)/2} 0 0" rpy="0 0 0" />
         <geometry name="${name}_shoulder_lift_visual_geom">
-          <box size="${ax12_height+arm_major_length} ${ax12_width} ${ax12_depth}"/>
+          <box size="${ax12_center+arm_major_length} ${ax12_width} ${ax12_depth}"/>
         </geometry>
         <material name="Orange" />
@@ -58,7 +59,7 @@
     <link name="${name}_elbow_flex_link">
       <visual name="${name}_elbow_flex_visual">
-        <origin xyz="${(ax12_height+arm_major_length)/2} 0 0" rpy="0 0 0" />
+        <origin xyz="${(ax12_center+arm_major_length)/2} 0 0" rpy="0 0 0" />
         <geometry name="${name}_elbow_flex_visual_geom">
-          <box size="${ax12_height+arm_major_length} ${ax12_width} ${ax12_depth}"/>
+          <box size="${ax12_center+arm_major_length} ${ax12_width} ${ax12_depth}"/>
         </geometry>
         <material name="Black" />
@@ -70,5 +71,5 @@
       <axis xyz="0 1 0" />
       <limit lower="-1.57" upper="1.57" effort="5.0" velocity="5" />
-      <origin xyz="0.125 0 0" rpy="0 0 0" />
+      <origin xyz="${ax12_center+arm_major_length} 0 0" rpy="0 0 0" />
       <parent link="${name}_elbow_flex_link"/>
       <child link="${name}_wrist_flex_link"/>

File: mini_max/mini_max_defs/urdf/gripper.urdf.xacro (robot description, xacro)
@@ -2,4 +2,21 @@
 <robot>
   <macro name="mini_gripper" params="name parent">
+    <!-- Palm -->
+    <joint name="${name}_palm_joint" type="fixed">
+      <axis xyz="0 0 1" />
+      <origin xyz="0.04 0 0" rpy="0 0 0" />
+      <parent link="${parent}_link"/>
+      <child link="${name}_palm_link"/>
+    </joint>
+    <link name="${name}_palm_link">
+      <visual name="${name}_palm_visual">
+        <origin xyz="0 0.005 0" rpy="0 0 0"/>
+        <geometry name="${name}_palm_visual_geom">
+          <box size="0.03 ${0.0375+0.0275} ${ax12_depth*1.1}"/>
+        </geometry>
+        <material name="Black" />
+      </visual>
+      <!-- TODO: add collision -->
+    </link>
     <!-- Static Side -->
     <joint name="${name}_static_joint" type="fixed">
@@ -11,5 +28,5 @@
     <link name="${name}_link">
       <visual name="${name}_static_visual">
-        <origin xyz="-0.05 0.025 0" rpy="-1.57 0 0"/>
+        <origin xyz="-0.06 0.0375 0" rpy="-1.57 0 0"/>
         <geometry name="${name}_static_visual_geom">
           <mesh filename="package://mini_max_defs/meshes/gripper.stl" />
@@ -22,5 +39,5 @@
     <joint name="${name}_joint" type="revolute">
       <axis xyz="0 0 1" />
-      <origin xyz="0.05 -0.025 0" rpy="0 0 0" />
+      <origin xyz="0.04 -0.0275 0" rpy="0 0 0" />
       <limit lower="-1.57"  upper="1.57" effort="5.0" velocity="5" />
       <parent link="${parent}_link"/>

File: mini_max/mini_max_defs/urdf/mini_max.urdf.xacro (robot description, xacro)
@@ -10,4 +10,10 @@
   <property name="ax12_depth" value="0.0318" />
   <property name="ax12_center" value="0.0385" />
+  <property name="calib_cam_x" value="0.010" />
+  <property name="calib_cam_y" value="0.000" />
+  <property name="calib_cam_z" value="0.025" />
+  <property name="calib_cam_rr" value="0.000" />
+  <property name="calib_cam_rp" value="0.080" />
+  <property name="calib_cam_ry" value="0.000" />
   <include filename="$(find mini_max_defs)/urdf/arm.urdf.xacro" />
   <include filename="$(find mini_max_defs)/urdf/gripper.urdf.xacro" />
@@ -80,5 +86,5 @@
      <parent link="head_pan_link" />
      <child link="head_tilt_link" />
-     <origin xyz="0 0 ${ax12_height+0.00635}" />
+     <origin xyz="0 0 ${ax12_center}" />
      <axis xyz="0 1.0 0"/>
      <limit effort="30" velocity="1.0" lower="-1.57" upper="1.57" />
@@ -96,5 +102,5 @@
   <!-- Head sensor frame -->
   <joint name="head_sensor_frame_joint" type="fixed">
-    <origin xyz="0 0 ${neck_height}" rpy="0 0 0" />
+    <origin xyz="${calib_cam_z} ${calib_cam_y} ${neck_height+calib_cam_x}" rpy="${calib_cam_rr} ${calib_cam_rp} ${calib_cam_ry}" />
     <parent link="head_tilt_link"/>
     <child link="head_sensor_frame"/>
@@ -102,5 +108,5 @@
   <link name="head_sensor_frame">
     <visual>
-      <origin xyz="-0.0254 0 0" rpy="0 0 -1.57" />
+      <origin xyz="${-calib_cam_z-0.0254} 0 0" rpy="0.0 0 -1.57" />
       <geometry>
         <mesh filename="package://mini_max_defs/meshes/kinect.stl" />

Commit message: (mini_max_defs) update for calibration

File: mini_max/mini_max_defs/urdf/arm.urdf.xacro (robot description, xacro)
@@ -3,5 +3,4 @@
   <!-- size properties -->
   <property name="arm_pan_height" value="0.00635" />
-  <!--<property name="arm_major_length" value="0.09208" />-->
   <property name="arm_major_length" value="0.06627" />
   <macro name="mini_arm" params="name parent *origin">
@@ -16,5 +15,5 @@
     <joint name="${name}_shoulder_pan_joint" type="revolute">
       <axis xyz="0 0 1" />
-      <origin xyz="0 0 0" rpy="0 0 0"/>
+      <origin xyz="0 0 0" rpy="0 0 ${shoulder_pan_offset}"/>
       <parent link="${name}_base_link"/>
       <child link="${name}_shoulder_pan_link"/>
@@ -35,12 +34,12 @@
       <axis xyz="0 1 0"/>
       <limit lower="-0.2" upper="2.617" effort="5.0" velocity="5" />
-      <origin xyz="0 0 ${ax12_center+arm_pan_height}" rpy="0 -1.57 0" />
+      <origin xyz="0 0 ${ax12_center+arm_pan_height}" rpy="0 -1.57 ${shoulder_lift_offset}" />
       <parent link="${name}_shoulder_pan_link"/>
       <child link="${name}_shoulder_lift_link"/>
     </joint>
     <link name="${name}_shoulder_lift_link">
-      <visual name="${name}_shoulder_lift_visual">
+      <visual>
         <origin xyz="${(ax12_center+arm_major_length)/2} 0 0" rpy="0 0 0" />
-        <geometry name="${name}_shoulder_lift_visual_geom">
+        <geometry>
           <box size="${ax12_center+arm_major_length} ${ax12_width} ${ax12_depth}"/>
         </geometry>
@@ -53,12 +52,12 @@
       <axis xyz="0 1 0" />
       <limit lower="-1.57" upper="2.617" effort="5.0" velocity="5" />
-      <origin xyz="${ax12_center+arm_major_length} 0 0" rpy="0 0 0" />
+      <origin xyz="${ax12_center+arm_major_length} 0 0" rpy="0 ${elbow_flex_offset} 0" />
       <parent link="${name}_shoulder_lift_link"/>
       <child link="${name}_elbow_flex_link"/>
     </joint>
     <link name="${name}_elbow_flex_link">
-      <visual name="${name}_elbow_flex_visual">
+      <visual>
         <origin xyz="${(ax12_center+arm_major_length)/2} 0 0" rpy="0 0 0" />
-        <geometry name="${name}_elbow_flex_visual_geom">
+        <geometry>
           <box size="${ax12_center+arm_major_length} ${ax12_width} ${ax12_depth}"/>
         </geometry>
@@ -71,13 +70,12 @@
       <axis xyz="0 1 0" />
       <limit lower="-1.57" upper="1.57" effort="5.0" velocity="5" />
-      <origin xyz="${ax12_center+arm_major_length} 0 0" rpy="0 0 0" />
+      <origin xyz="${ax12_center+arm_major_length} 0 0" rpy="${wrist_flex_offset} 0 0" />
       <parent link="${name}_elbow_flex_link"/>
       <child link="${name}_wrist_flex_link"/>
     </joint>
     <link name="${name}_wrist_flex_link">
-      <visual name="${name}_wrist_flex_visual">
+      <visual>
         <origin xyz="${0.050/2} 0 0" rpy="0 0 0" />
-        <geometry name="${name}_wrist_flex_visual_geom">
-          <!--<mesh filename="package://pr2_defs/meshes/wrist_flex.stl" />-->
+        <geometry>
           <box size="0.05 0.050 ${ax12_depth}"/>
         </geometry>

File: mini_max/mini_max_defs/urdf/mini_max.urdf.xacro (robot description, xacro)
@@ -10,10 +10,5 @@
   <property name="ax12_depth" value="0.0318" />
   <property name="ax12_center" value="0.0385" />
-  <property name="calib_cam_x" value="0.010" />
-  <property name="calib_cam_y" value="0.000" />
-  <property name="calib_cam_z" value="0.025" />
-  <property name="calib_cam_rr" value="0.000" />
-  <property name="calib_cam_rp" value="0.080" />
-  <property name="calib_cam_ry" value="0.000" />
+  <include filename="$(find mini_max_defs)/urdf/calibration.urdf.xacro" />
   <include filename="$(find mini_max_defs)/urdf/arm.urdf.xacro" />
   <include filename="$(find mini_max_defs)/urdf/gripper.urdf.xacro" />
@@ -70,6 +65,6 @@
      <parent link="column_link" />
      <child link="head_pan_link" />
-     <origin xyz="0 0 0"/>
      <axis xyz="0 0 1.0"/>
+     <origin xyz="0 0 0" rpy="0 0 ${head_pan_offset}"/>
      <limit effort="30" velocity="1.0" lower="-1.57" upper="1.57" />
   </joint>
@@ -87,5 +82,5 @@
      <child link="head_tilt_link" />
      <origin xyz="0 0 ${ax12_center}" />
-     <axis xyz="0 1.0 0"/>
+     <axis xyz="0 1.0 0" rpy="0 ${head_tilt_offset} 0" />
      <limit effort="30" velocity="1.0" lower="-1.57" upper="1.57" />
   </joint>
@@ -102,5 +97,5 @@
   <!-- Head sensor frame -->
   <joint name="head_sensor_frame_joint" type="fixed">
-    <origin xyz="${calib_cam_z} ${calib_cam_y} ${neck_height+calib_cam_x}" rpy="${calib_cam_rr} ${calib_cam_rp} ${calib_cam_ry}" />
+    <origin xyz="${calib_cam_x} ${calib_cam_y} ${neck_height+calib_cam_z}" rpy="${calib_cam_rr} ${calib_cam_rp} ${calib_cam_ry}" />
     <parent link="head_tilt_link"/>
     <child link="head_sensor_frame"/>
@@ -108,5 +103,5 @@
   <link name="head_sensor_frame">
     <visual>
-      <origin xyz="${-calib_cam_z-0.0254} 0 0" rpy="0.0 0 -1.57" />
+      <origin xyz="${-calib_cam_x-0.0254} 0 0" rpy="0.0 0 -1.57" />
       <geometry>
         <mesh filename="package://mini_max_defs/meshes/kinect.stl" />
