Commit message: (mini_max) move mini_max branch into electric tree

File: mini_max/mini_max_defs/urdf/mini_max.urdf.xacro (robot description, xacro)
@@ -6,40 +6,46 @@
   <property name="body_height" value="0.3302" />
   <property name="neck_height" value="0.0857" />
-  <property name="ax12_height" value="0.04762" />
-  <property name="ax12_width" value="0.0381" />
-  <property name="ax12_depth" value="0.0318" />
-  <property name="ax12_center" value="0.0385" />
-  <include filename="$(find mini_max_defs)/urdf/calibration.urdf.xacro" />
-  <include filename="$(find mini_max_defs)/urdf/arm.urdf.xacro" />
-  <include filename="$(find mini_max_defs)/urdf/gripper.urdf.xacro" />
+  <include filename="$(find turtlebot_arm_description)/urdf/arm.xacro" />
   <!-- colors -->
-  <material name="Black">
-    <color rgba="0.2 0.2 0.2 1.0"/>
-  </material>
-  <material name="Orange">
-    <color rgba="1.0  0.55 0.0 1.0"/>
-  </material>
-  <material name="Grey">
+  <material name="grey">
     <color rgba="0.7 0.7 0.7 1.0"/>
   </material>
   <!-- create base -->
-  <property name="create_radius" value="0.1778" />
-  <property name="create_height" value="0.0762" />
+  <property name="create_radius" value="0.16495" />
+  <property name="create_height" value="0.0611632" />
+  <link name="base_footprint">
+    <inertial>
+      <mass value="0.0001" />
+      <origin xyz="0 0 0" />
+      <inertia ixx="0.0001" ixy="0.0" ixz="0.0"
+              iyy="0.0001" iyz="0.0"
+              izz="0.0001" />
+    </inertial>
+  </link>
+  <joint name="base_footprint_joint" type="fixed">
+    <origin xyz="0 0 0.017" rpy="0 0 0" />
+    <parent link="base_footprint"/>
+    <child link="base_link" />
+  </joint>
   <link name="base_link">
+    <inertial>
+      <mass value="1" />
+      <origin xyz="0 0 0.0308" />
+      <inertia ixx="1.0" ixy="0.0" ixz="0.0"
+        iyy="1.0" iyz="0.0" izz="1.0" />
+    </inertial>
     <visual>
-      <origin xyz="0 0 ${create_height/2}" rpy="0 0 0" />
+      <origin xyz=" 0 0 0.0308" rpy="0 0 0" />
       <geometry>
-        <cylinder radius="${create_radius}" length="${create_height}" />
+        <mesh filename="package://turtlebot_description/meshes/create_body.dae"/>
       </geometry>
-      <material name="Grey" />
     </visual>
     <collision>
-      <origin xyz="0 0 ${create_height/2}" rpy="0 0 0" />
+      <origin xyz="0.0 0.0 0.0308" rpy="0 0 0" />
       <geometry>
-        <cylinder radius="${create_radius}" length="${create_height}" />
+        <cylinder length="0.0611632" radius="0.16495"/>
       </geometry>
     </collision>
   </link>
-  <!-- head w/ kinect, pan/tilt -->
   <joint name="column_joint" type="fixed">
     <parent link="base_link" />
@@ -53,5 +59,5 @@
         <mesh filename="package://mini_max_defs/meshes/body.stl"  />
       </geometry>
-      <material name="Black" />
+      <material name="black" />
     </visual>
     <collision>
@@ -62,57 +68,43 @@
     </collision>
   </link>
-  <joint name="head_pan_joint" type="revolute">
-     <parent link="column_link" />
-     <child link="head_pan_link" />
-     <axis xyz="0 0 1.0"/>
-     <origin xyz="0 0 0" rpy="0 0 ${head_pan_offset}"/>
-     <limit effort="30" velocity="1.0" lower="-1.57" upper="1.57" />
-  </joint>
-  <link name="head_pan_link">
-    <visual>
-      <origin xyz="0 0 ${(ax12_height+0.00635)/2}"/>
-      <geometry>
-        <box size="${ax12_depth} ${ax12_width} ${ax12_height+0.00635}"/>
-      </geometry>
-      <material name="Orange"/>
-    </visual>
-  </link>
-  <joint name="head_tilt_joint" type="revolute">
-     <parent link="head_pan_link" />
-     <child link="head_tilt_link" />
-     <origin xyz="0 0 ${ax12_center}" />
-     <axis xyz="0 1.0 0" rpy="0 ${head_tilt_offset} 0" />
-     <limit effort="30" velocity="1.0" lower="-1.57" upper="1.57" />
-  </joint>
-  <link name="head_tilt_link">
-    <visual>
-      <origin xyz="0 0 ${neck_height/2}"/>
-      <geometry>
-        <box size=".0381 .0381 ${neck_height}"/>
-      </geometry>
-      <material name="Black"/>
-    </visual>
-    <!-- TODO: add collision -->
-  </link>
-  <!-- Head sensor frame -->
+  <!-- head w/ kinect, pan/tilt -->
+  <bioloid_F3_revolute parent="column_link" name="head_pan" color="white" vlimit="1.571" llimit="-2.0" ulimit="2.0">
+    <origin xyz="0 0 0" rpy="${M_PI} 0 ${M_PI}"/>
+  </bioloid_F3_revolute>
+  <dynamixel_AX12_fixed parent="head_pan_link" name="head_pan_servo">
+    <origin xyz="0 0 ${-AX12_HEIGHT-F10_HEIGHT+0.001}" rpy="0 ${M_PI} 0"/>
+  </dynamixel_AX12_fixed>
+  <bioloid_F2_revolute parent="head_pan_servo_link" name="head_tilt" color="white" vlimit="1.571" llimit="-2.671" ulimit="2.671">
+    <origin xyz="0 0 0" rpy="0 0 0"/>
+  </bioloid_F2_revolute>
   <joint name="head_sensor_frame_joint" type="fixed">
-    <origin xyz="${calib_cam_x} ${calib_cam_y} ${neck_height+calib_cam_z}" rpy="${calib_cam_rr} ${calib_cam_rp} ${calib_cam_ry}" />
-    <parent link="head_tilt_link"/>
-    <child link="head_sensor_frame"/>
+    <origin xyz="0.03 0 0.075" rpy="0 0 0" />
+    <parent link="head_tilt_link" />
+    <child link="head_sensor_frame" />
   </joint>
   <link name="head_sensor_frame">
+    <inertial>
+      <mass value="0.00001" />
+      <origin xyz="0 0 0" />
+      <inertia ixx="1.0" ixy="0.0" ixz="0.0"
+        iyy="1.0" iyz="0.0"
+        izz="1.0" />
+    </inertial>
     <visual>
-      <origin xyz="${-calib_cam_x-0.0254} 0 0" rpy="0.0 0 -1.57" />
+      <origin xyz=" 0 0 0 " rpy="0 0 0" />
       <geometry>
-        <mesh filename="package://mini_max_defs/meshes/kinect.stl" />
+        <mesh filename="package://turtlebot_description/meshes/kinect.dae"/>
       </geometry>
-      <material name="Black" />
     </visual>
-    <!-- TODO: add collision -->
+    <collision>
+      <origin xyz="0.0 0.0 0.0" rpy="0 0 0" />
+      <geometry>
+        <box size="0.0730 .2760 0.0720"/>
+      </geometry>
+    </collision>
   </link>
   <!-- add arm and gripper -->
-  <mini_arm name="arm" parent="base">
+  <turtlebot_arm parent="base_link" color="white" gripper_color="grey">
     <origin xyz="0.104775 -0.0381 ${create_height+standoff_height+material_thickness}"/>
-  </mini_arm>
-  <mini_gripper name="gripper" parent="arm_wrist_flex"/>
+  </turtlebot_arm>
 </robot>
