Commit message: (maxwell) updates to urdf, merge in max_lite

File: maxwell/max_lite/urdf/max_lite.urdf.xacro (robot description, xacro)
@@ -1,4 +1,4 @@
 <?xml version="1.0"?>
-<robot name="maxwell" >
+<robot name="max_lite" >
   <property name='calib_cam_x' value='0.00259672' />
   <property name='calib_cam_y' value='0.0307021' />
@@ -10,14 +10,14 @@
   <property name="column_height" value="1.171575" /> <!-- deck to top of 80/20: 46-1/8" -->
   <include filename="$(find maxwell_defs)/urdf/hardware/ax12.xacro" />
-  <include filename="$(find maxwell_defs)/urdf/hardware/rx64.xacro" />
+  <include filename="$(find maxwell_defs)/urdf/hardware/rx28.xacro" />
   <!-- The following included files set up definitions of parts of the robot body -->
   <include filename="$(find maxwell_defs)/urdf/base.urdf.xacro" />
   <include filename="$(find maxwell_defs)/urdf/torso.urdf.xacro" />
-  <include filename="$(find maxwell_defs)/urdf/arm.urdf.xacro" />
   <include filename="$(find maxwell_defs)/urdf/gripper.urdf.xacro" />
   <include filename="$(find maxwell_defs)/urdf/head.urdf.xacro" />
   <include filename="$(find maxwell_defs)/urdf/materials.urdf.xacro" />
-  <!-- Now we can start using the macros included above to define the actual Maxwell -->
-  <armadillo_base name="base" color="Orange"/>
+  <include filename="$(find max_lite)/urdf/arm_lite.urdf.xacro" />
+  <!-- Now we can start using the macros included above to define the actual Max Lite -->
+  <armadillo_base name="base" color="Blue"/>
   <!-- Add Torso Upright -->
   <maxwell_torso name="torso" parent="base">
@@ -25,13 +25,13 @@
   </maxwell_torso>
   <!-- Arm -->
-  <maxwell_arm name="arm" parent="torso">
-    <origin xyz="0.0611 0 ${arm_height}"/>
-  </maxwell_arm>
+  <max_lite_arm name="arm" parent="torso">
+    <origin xyz="0.0513 0 ${arm_height}"/>
+  </max_lite_arm>
   <!-- Gripper -->
-  <maxwell_gripper name="gripper" parent="arm_wrist_roll" color="Orange">
+  <maxwell_gripper name="gripper" parent="arm_wrist_roll" color="Blue">
     <origin xyz="0 0 0" />
   </maxwell_gripper>
   <!-- Head -->
-  <maxwell_head name="head" parent="torso" color="Orange">
+  <maxwell_head name="head" parent="torso" color="Blue">
     <origin xyz="0 0 ${column_height}"/>
   </maxwell_head>

File: maxwell/maxwell_defs/urdf/base.urdf.xacro (robot description, xacro)
@@ -15,5 +15,5 @@
   <property name="base_laser_z" value="0.1885" />
   <!-- define a wheel -->
-  <macro name="armadillo_wheel" params="suffix parent reflect">
+  <macro name="armadillo_wheel" params="suffix parent reflect color">
     <joint name="${parent}_${suffix}_wheel_joint" type="continuous">
       <axis xyz="0 0 1" />
@@ -30,10 +30,10 @@
           <cylinder radius="${wheel_radius}" length="${wheel_length}"/>
         </geometry>
-        <material name="Orange" />
+        <material name="${color}" />
       </visual>
     </link>
   </macro>
   <!-- The xacro macro armadillo_base contains: base and wheels -->
-  <macro name="armadillo_base" params="name">
+  <macro name="armadillo_base" params="name color">
     <link name="${name}_link">
       <visual>
@@ -56,6 +56,6 @@
     </hokuyo_urg_laser>
     <!-- drive wheels -->
-    <armadillo_wheel parent="${name}" suffix="l" reflect="1" />
-    <armadillo_wheel parent="${name}" suffix="r" reflect="-1" />
+    <armadillo_wheel parent="${name}" suffix="l" reflect="1" color="${color}"/>
+    <armadillo_wheel parent="${name}" suffix="r" reflect="-1" color="${color}"/>
   </macro>
 </robot>

File: maxwell/maxwell_defs/urdf/gripper.urdf.xacro (robot description, xacro)
@@ -1,5 +1,5 @@
 <?xml version="1.0"?>
 <robot>
-  <macro name="maxwell_gripper" params="name parent *origin">
+  <macro name="maxwell_gripper" params="name parent color *origin">
     <ax12_F6_fixed parent="${parent}_link" name="${name}_F6_1" color="Black">
       <origin xyz="${0.0381/2} 0.017 -0.014" rpy="0 0 0"/>
@@ -26,8 +26,8 @@
       <origin xyz="0 0 -0.042" rpy="1.57 1.57 0"/>
     </dynamixel_ax12_pan>
-    <ax12_F1_revolute parent="left_${name}_servo_link" name="l_${name}" llimit="-1.57" ulimit="1.57" vlimit="0.5" color="Orange">
+    <ax12_F1_revolute parent="left_${name}_servo_link" name="l_${name}" llimit="-1.57" ulimit="1.57" vlimit="0.5" color="${color}">
       <origin xyz="0 0 0" rpy="3.14 0 1.57"/>
     </ax12_F1_revolute>
-    <ax12_F1_revolute parent="right_${name}_servo_link" name="r_${name}" llimit="-1.57" ulimit="1.57" vlimit="0.5" color="Orange">
+    <ax12_F1_revolute parent="right_${name}_servo_link" name="r_${name}" llimit="-1.57" ulimit="1.57" vlimit="0.5" color="${color}">
       <origin xyz="0 0 0" rpy="0 0 -1.57"/>
     </ax12_F1_revolute>

File: maxwell/maxwell_defs/urdf/head.urdf.xacro (robot description, xacro)
@@ -25,5 +25,5 @@
   </macro>
   <!-- origin is center of head tilt rotation -->
-  <macro name="maxwell_head" params="name parent *origin">
+  <macro name="maxwell_head" params="name parent color *origin">
     <joint name="${name}_joint" type="fixed">
       <insert_block name="origin" />
@@ -42,5 +42,5 @@
       <origin xyz="0.010 0 0.0254" rpy="0 0 0"/>
     </dynamixel_ax12_pan>
-    <ax12_side_revolute parent="${name}_pan_servo_link" name="${name}_pan" llimit="-2.617" ulimit="2.617" vlimit="1.0" color="Orange">
+    <ax12_side_revolute parent="${name}_pan_servo_link" name="${name}_pan" llimit="-2.617" ulimit="2.617" vlimit="1.0" color="${color}">
       <origin xyz="0 0 ${AX12_WIDTH/2}" rpy="0 0 0"/>
     </ax12_side_revolute>
@@ -55,5 +55,5 @@
       <origin xyz="0 0 ${AX12_HEIGHT+0.003}" rpy="0 0 0"/>
     </dynamixel_ax12_tilt>
-    <ax12_hinge_revolute parent="${name}_tilt_servo_link" name="${name}_tilt" llimit="-2.617" ulimit="2.617" vlimit="1.0" color="Orange">
+    <ax12_hinge_revolute parent="${name}_tilt_servo_link" name="${name}_tilt" llimit="-2.617" ulimit="2.617" vlimit="1.0" color="${color}">
      <origin xyz="0 0 0" rpy="0 0 0"/>
     </ax12_hinge_revolute>

File: maxwell/maxwell_defs/urdf/materials.urdf.xacro (robot description, xacro)
@@ -16,3 +16,6 @@
     <color rgba="1.0 1.0 1.0 1.0"/>
   </material>
+  <material name="Blue">
+    <color rgba="0.0 0.0 0.8 1.0"/>
+  </material>
 </robot>
