Commit message: (maxwell_defs) reworking meshes

File: maxwell/maxwell_defs/urdf/head.urdf.xacro (robot description, xacro)
@@ -1,55 +1,87 @@
 <?xml version="1.0"?>
 <robot>
+  <property name="M_PI" value="3.14159"/>
+  <property name="AX12_WIDTH" value="0.038"/>
+  <property name="AX12_HEIGHT" value="0.0385"/>
+  <property name="F10_HEIGHT" value="0.004"/>
+  <include filename="$(find maxwell_defs)/urdf/hardware/bioloid_ax12.xacro" />
+  <include filename="$(find maxwell_defs)/urdf/hardware/bioloid_F2_revolute.xacro" />
+  <include filename="$(find maxwell_defs)/urdf/hardware/bioloid_F3_revolute.xacro" />
+  <include filename="$(find maxwell_defs)/urdf/hardware/bioloid_F3_fixed.xacro" />
   <!-- origin is center of head tilt rotation -->
   <macro name="maxwell_head" params="name parent *origin">
     <!-- Head pan -->
-    <joint name="${name}_pan_joint" type="revolute">
-      <axis xyz="0 0 1" />
+    <joint name="${name}_pan_servo_joint" type="fixed">
       <insert_block name="origin" />
-      <parent link="${parent}_link"/>
-      <child link="${name}_pan_link"/>
-      <limit lower="-2.617" upper="2.617" effort="1" velocity="1" />
+      <parent link="${parent}"/>
+      <child link="${name}_pan_servo_link" />
     </joint>
-    <link name="${name}_pan_link">
+    <link name="${name}_pan_servo_link">
+      <inertial>
+        <mass value="0.00001" />
+        <origin xyz="0 0 0" />
+        <inertia ixx="1.0" ixy="0.0" ixz="0.0"
+          iyy="1.0" iyz="0.0"
+          izz="1.0" />
+      </inertial>
       <visual>
-        <origin xyz="0 0 ${0.0635/2}" rpy="0 0 0 " />
+        <origin xyz="0 0 0" rpy="1.57 0 1.57" />
         <geometry>
-          <box size="${ax12_depth} ${ax12_width} ${ax12_height+0.00635}"/>
+          <mesh filename="package://maxwell_defs/meshes/ax12_box.stl" scale="0.001 0.001 0.001"/>
         </geometry>
-        <material name="Black" />
+        <material name="Black"/>
       </visual>
       <collision>
-        <origin xyz="0 0 ${0.0635/2}" rpy="0 0 0 " />
+        <origin xyz="-0.01241 0.0 0.0" rpy="1.57 0 1.57" />
         <geometry>
-          <box size="${ax12_depth} ${ax12_width} ${ax12_height+0.00635}"/>
+          <box size="0.025 0.038 0.04762"/>
         </geometry>
       </collision>
     </link>
-    <!-- Head tilt -->
-    <joint name="${name}_tilt_joint" type="revolute">
-      <axis xyz="0 1 0" />
-      <limit lower="-1.57" upper="1.57" effort="5.0" velocity="5" />
-      <origin xyz="0 0 0" rpy="0 0 0" />
-      <parent link="${name}_pan_link"/>
-      <child link="${name}_tilt_link"/>
+    <joint name="${name}_pan_joint" type="revolute">
+      <origin xyz="0 0 ${AX12_WIDTH/2}"/>
+      <axis xyz="0 0 1"/>
+      <limit effort="30" velocity="1.0" lower="-2.61799388" upper="2.61799388" />
+      <parent link="${name}_pan_servo_link"/>
+      <child link="${name}_pan_link" />
     </joint>
-    <link name="${name}_tilt_link">
+    <link name="${name}_pan_link">
+      <inertial>
+        <mass value="0.00001" />
+        <origin xyz="0 0 0" />
+        <inertia ixx="1.0" ixy="0.0" ixz="0.0"
+          iyy="1.0" iyz="0.0"
+          izz="1.0" />
+      </inertial>
       <visual>
-        <origin xyz="0 0 ${0.0381/2}" rpy="0.0 0.0 0.0" />
+        <origin xyz=" 0 0 0 " rpy="3.14 0 0" />
         <geometry>
-          <box size=".0381 .0381 .0381"/>
+          <mesh filename="package://maxwell_defs/meshes/F3.stl" scale="0.001 0.001 0.001"/>
         </geometry>
-        <material name="Orange" />
+        <material name="Black"/>
       </visual>
       <collision>
-        <origin xyz="0 0 ${0.0381/2}" rpy="0.0 0.0 0.0" />
+        <origin xyz="0.0 0.0 0.0045" rpy="0 0 0" />
         <geometry>
-          <box size=".0381 .0381 .0381"/>
+          <box size="0.025 0.038 0.009"/>
         </geometry>
       </collision>
     </link>
+    <bioloid_F3_fixed parent="${name}_pan_servo_link" name="${name}_tilt_left_side" joint_name="${name}_tilt_left_joint" color="Black">
+      <origin xyz="-0.015 ${-AX12_WIDTH/2} 0" rpy="1.57 0 0"/>
+    </bioloid_F3_fixed>
+    <bioloid_F3_fixed parent="${name}_pan_servo_link" name="${name}_tilt_right_side" joint_name="${name}_tilt_right_joint" color="Black">
+      <origin xyz="-0.015 ${AX12_WIDTH/2} 0" rpy="-1.57 0 0"/>
+    </bioloid_F3_fixed>
+    <!-- Head tilt -->
+    <bioloid_ax12 parent="${name}_pan_link" name="${name}_tilt_servo" color="Black">
+      <origin xyz="0 0 ${AX12_HEIGHT+F10_HEIGHT-0.001}" rpy="0 0 0"/>
+    </bioloid_ax12>
+    <bioloid_F2_revolute parent="${name}_tilt_servo_link" name="${name}_tilt" joint_name="${name}_tilt_joint" color="Orange">
+     <origin xyz="0 0 0" rpy="0 0 0"/>
+    </bioloid_F2_revolute>
     <!-- Head sensor frame -->
     <joint name="${name}_sensor_frame_joint" type="fixed">
-      <origin xyz="${calib_cam_x} ${calib_cam_y} ${calib_cam_z}" rpy="${calib_cam_rr} ${calib_cam_rp} ${calib_cam_ry}" />
+      <origin xyz="0 0 0.0425"/>
       <parent link="${name}_tilt_link"/>
       <child link="${name}_sensor_frame"/>
@@ -57,5 +89,5 @@
     <link name="${name}_sensor_frame">
       <visual>
-        <origin xyz="${-calib_cam_x-0.0254} 0 0" rpy="0 0 -1.57" />
+        <origin xyz="-0.03 0 0" rpy="0 0 -1.57" />
         <geometry>
           <mesh filename="package://maxwell_defs/meshes/kinect.stl" />
@@ -63,5 +95,12 @@
         <material name="Black" />
       </visual>
-    </link> <!-- comment this link out for calibration -->
+    </link>
+    <!-- Openni Link -->
+    <joint name="openni_camera_joint" type="fixed">
+      <origin xyz="${calib_cam_x} ${calib_cam_y} ${calib_cam_z}" rpy="${calib_cam_rr} ${calib_cam_rp} ${calib_cam_ry}" />
+      <parent link="${name}_sensor_frame"/>
+      <child link="openni_camera"/>
+    </joint>
+    <link name="openni_camera"/>
   </macro>
 </robot>

File: maxwell/maxwell_defs/urdf/maxwell.urdf.xacro (robot description, xacro)
@@ -1,23 +1,8 @@
 <?xml version="1.0"?>
 <robot name="maxwell" >
-  <!-- Calibration from 8/7
-  <property name='calib_cam_x' value='-0.000859868' />
-  <property name='calib_cam_y' value='0.0171667' />
-  <property name='calib_cam_z' value='0.0192186' />
-  <property name='calib_cam_rr' value='-0.0432624' />
-  <property name='calib_cam_rp' value='-0.0226177' />
-  <property name='calib_cam_ry' value='0.00714413' />
-  -->
-  <!-- Calibration from 8/8
-  <property name='calib_cam_x' value='-0.00515338' />
-  <property name='calib_cam_y' value='0.0131489' />
-  <property name='calib_cam_z' value='0.0169829' />
-  <property name='calib_cam_rr' value='-0.0397998' />
-  <property name='calib_cam_rp' value='-0.0241423' />
-  <property name='calib_cam_ry' value='0.00627637' />
-  -->
   <property name='calib_cam_x' value='0.00468423' />
   <property name='calib_cam_y' value='0.0060704' />
-  <property name='calib_cam_z' value='0.0118428' />
+  <property name='calib_cam_z' value='-0.0306572' />
+  <!--<property name='calib_cam_z' value='0.0118428' />-->
   <property name='calib_cam_rr' value='-0.024976' />
   <property name='calib_cam_rp' value='-0.0119664' />
@@ -36,7 +21,8 @@
   <property name="ax12_center" value="0.0385" />
   <!-- height properties -->
-  <!--<property name="arm_height" value="0.911225" />-->
-  <property name="arm_height" value="0.885825" /><!-- height to shoulder lift rotation -->
-  <property name="column_height" value="1.397" /> <!-- height to neck tilt rotation -->
+  <!--<property name="arm_height" value="0.885825" /> height to shoulder lift rotation -->
+   <!--<property name="column_height" value="1.397" /> height to neck tilt rotation -->
+  <property name="arm_height" value="0.5921375" /> <!-- deck to bottom of arm mount TODO: update this -->
+  <property name="column_height" value="1.171575" /> <!-- deck to top of 80/20: 46-1/8" -->
   <!-- The following included files set up definitions of parts of the robot body -->
   <include filename="$(find maxwell_defs)/urdf/base.urdf.xacro" />
@@ -50,9 +36,9 @@
   <!-- Add Torso Upright -->
   <maxwell_torso name="torso" parent="base">
-    <origin xyz="-0.00635 0 ${arm_height}"/>
+    <origin xyz="-0.00635 0 ${base_size_z}"/>
   </maxwell_torso>
   <!-- Arm -->
   <maxwell_arm name="arm" parent="torso">
-    <origin xyz="0.0608 0 0"/>
+    <origin xyz="0.0608 0 ${arm_height+.15}"/>
   </maxwell_arm>
   <!-- Gripper -->
@@ -61,7 +47,8 @@
   </maxwell_gripper>
   <!-- Kinect head -->
-  <maxwell_head name="head" parent="base">
+  <maxwell_head name="head" parent="torso_link">
     <!--<origin xyz="0.0157 0 ${column_height}"/>-->
-    <origin xyz="${0.0157+0.05715/2} -0.005 ${column_height}"/>
+    <!--<origin xyz="${0.0157+0.05715/2} -0.005 ${column_height+0.0460375}"/>-->
+    <origin xyz="0 0 ${column_height+0.0270375}"/>
   </maxwell_head>
 </robot>

File: maxwell/maxwell_defs/urdf/sensors/hokuyo_urg_laser.urdf.xacro (robot description, xacro)
@@ -1,5 +1,5 @@
 <?xml version="1.0"?>
-<robot xmlns:xacro="http://ros.org/wiki/xacro">
-  <xacro:macro name="hokuyo_urg_laser" params="name parent *origin">
+<robot>
+  <macro name="hokuyo_urg_laser" params="name parent *origin">
     <joint name="${name}_joint" type="fixed">
       <axis xyz="0 1 0" />
@@ -28,4 +28,4 @@
       </collision>
     </link>
-  </xacro:macro>
+  </macro>
 </robot>

File: maxwell/maxwell_defs/urdf/torso.urdf.xacro (robot description, xacro)
@@ -10,5 +10,5 @@
     <link name="${name}_link">
       <visual>
-        <origin xyz="0 0 ${column_height/2-arm_height}" rpy="0 0 0 " />
+        <origin xyz="0 0 ${column_height/2}" rpy="0 0 0 " />
         <geometry>
           <box size="0.0254 0.0254 ${column_height}"/>
@@ -17,5 +17,5 @@
       </visual>
       <collision>
-        <origin xyz="0 0 ${column_height/2-arm_height}" rpy="0 0 0 " />
+        <origin xyz="0 0 ${column_height/2}" rpy="0 0 0 " />
         <geometry>
           <box size="0.0254 0.0254 ${column_height}"/>

Commit message: (maxwell_defs) update for calibration

File: maxwell/maxwell_defs/urdf/head.urdf.xacro (robot description, xacro)
@@ -65,5 +65,5 @@
     </joint>
     <link name="${name}_sensor_frame">
-      <visual>
+      <!--<visual>
         <origin xyz="-0.03 0 0" rpy="0 0 -1.57" />
         <geometry>
@@ -77,7 +77,7 @@
           <box size="0.064 0.28 0.04"/>
         </geometry>
-      </collision>
+      </collision>-->
     </link>
-    <!-- Openni Link -->
+    <!-- Openni Link
     <joint name="openni_camera_joint" type="fixed">
       <origin xyz="${calib_cam_x} ${calib_cam_y} ${calib_cam_z}" rpy="${calib_cam_rr} ${calib_cam_rp} ${calib_cam_ry}" />
@@ -85,5 +85,5 @@
       <child link="openni_camera"/>
     </joint>
-    <link name="openni_camera"/>
+    <link name="openni_camera"/>-->
   </macro>
 </robot>

File: maxwell/maxwell_defs/urdf/maxwell.urdf.xacro (robot description, xacro)
@@ -11,4 +11,5 @@
   <include filename="$(find maxwell_defs)/urdf/hardware/ax12.xacro" />
   <include filename="$(find maxwell_defs)/urdf/hardware/rx64.xacro" />
+  <include filename="$(find maxwell_defs)/urdf/sensors/kinect_camera.urdf.xacro" />
   <!-- The following included files set up definitions of parts of the robot body -->
   <include filename="$(find maxwell_defs)/urdf/base.urdf.xacro" />
@@ -36,3 +37,6 @@
     <origin xyz="0 0 ${column_height}"/>
   </maxwell_head>
+  <kinect_camera name="head_kinect" parent="head_sensor_frame">
+    <origin xyz="0 0 0"/>
+  </kinect_camera>
 </robot>
