Commit message: (maxwell_defs) move gripper frame

File: maxwell/maxwell_defs/urdf/gripper.urdf.xacro (robot description, xacro)
@@ -47,5 +47,5 @@
     <joint name="${name}_joint" type="fixed">
       <axis xyz="0 0 1" />
-      <origin xyz="0.16 0 0" rpy="0 0 0"/>
+      <origin xyz="0.15 0 -0.015" rpy="0 0 0"/>
       <parent link="${parent}_link"/>
       <child link="${name}_link"/>

Commit message: (maxwell_defs) add sphere to gripper link to avoid problem with collision objects in arm nav

File: maxwell/maxwell_defs/urdf/gripper.urdf.xacro (robot description, xacro)
@@ -51,5 +51,12 @@
       <child link="${name}_link"/>
     </joint>
-    <link name="${name}_link"/>
+    <link name="${name}_link">
+      <visual>
+        <origin xyz="0.0 0.0 0" rpy="0 0 0"/>
+        <geometry>
+          <sphere radius="0.0005"/>
+        </geometry>
+      </visual>
+    </link>
   </macro>
 </robot>
