Commit message: (maxwell_defs) add collision models

File: maxwell/maxwell_defs/urdf/arm.urdf.xacro (robot description, xacro)
@@ -18,5 +18,10 @@
         <material name="Black" />
       </visual>
-      <!-- TODO: add collision -->
+      <collision>
+        <origin xyz="${-0.065/2+0.0127} 0 0.040" rpy="0 0 0" />
+        <geometry>
+          <box size="0.065 0.057 0.120"/>
+        </geometry>
+      </collision>
     </link>
     <!-- Shoulder lift -->
@@ -36,5 +41,10 @@
         <material name="Grey" />
       </visual>
-      <!-- TODO: add collision -->
+      <collision>
+        <origin xyz="${0.165/2} 0 0" rpy="0 0 0" />
+        <geometry>
+          <box size="0.165 0.057 0.040"/>
+        </geometry>
+      </collision>
     </link>
     <!-- Elbow -->
@@ -49,5 +59,5 @@
       <visual name="${name}_elbow_flex_visual">
         <origin xyz="${0.125/2} 0 0" rpy="0 0 0" />
-        <geometry name="${name}_elbow_flex_visual_geom">
+        <geometry>
           <!--<mesh filename="package://pr2_defs/meshes/shoulder_yaw.stl" />-->
           <box size="0.125 0.057 0.040"/>
@@ -55,5 +65,10 @@
         <material name="Black" />
       </visual>
-      <!-- TODO: add collision -->
+      <collision>
+        <origin xyz="${0.125/2} 0 0" rpy="0 0 0" />
+        <geometry>
+          <box size="0.125 0.057 0.040"/>
+        </geometry>
+      </collision>
     </link>
     <!-- Wrist flex -->
@@ -74,5 +89,10 @@
         <material name="Grey" />
       </visual>
-      <!-- TODO: add collision -->
+      <collision>
+        <origin xyz="${0.030/2} 0 0" rpy="0 0 0" />
+        <geometry>
+          <box size="0.030 0.057 0.040"/>
+        </geometry>
+      </collision>
     </link>
     <!-- Wrist roll -->
@@ -93,5 +113,10 @@
         <material name="Black" />
       </visual>
-      <!-- TODO: add collision -->
+      <collision>
+        <origin xyz="0.05 0 0" rpy="0 0 0" />
+        <geometry>
+          <box size="0.100 0.065 0.050"/>
+        </geometry>
+      </collision>
     </link>
   </macro>

File: maxwell/maxwell_defs/urdf/gripper.urdf.xacro (robot description, xacro)
@@ -17,5 +17,10 @@
         <material name="Orange" />
       </visual>
-      <!-- TODO: add collision -->
+      <collision>
+        <origin xyz="0 0 0" rpy="0 0 0" />
+        <geometry>
+          <box size="0.125 0.01 0.03"/>
+        </geometry>
+      </collision>
     </link>
   </macro>

File: maxwell/maxwell_defs/urdf/head.urdf.xacro (robot description, xacro)
@@ -17,5 +17,10 @@
         <material name="Black" />
       </visual>
-      <!-- TODO: add collision -->
+      <collision>
+        <origin xyz="${-0.0635/4} 0 ${0.0381/2}" rpy="0 0 0" />
+        <geometry>
+          <box size=".0635 .0381 .0381"/>
+        </geometry>
+      </collision>
     </link>
     <!-- Head pan -->
@@ -35,5 +40,10 @@
         <material name="Black" />
       </visual>
-      <!-- TODO: add collision -->
+      <collision>
+        <origin xyz="0 0 ${0.0635/2}" rpy="0 0 0 " />
+        <geometry>
+          <box size=".0381 .0381 .0635"/>
+        </geometry>
+      </collision>
     </link>
     <!-- Head tilt -->
@@ -53,5 +63,10 @@
         <material name="Orange" />
       </visual>
-      <!-- TODO: add collision -->
+      <collision>
+        <origin xyz="0 0 ${0.0381/2}" rpy="0.0 0.0 0.0" />
+        <geometry>
+          <box size=".0381 .0381 .0381"/>
+        </geometry>
+      </collision>
     </link>
     <!-- Head sensor frame -->

Commit message: (maxwell_defs) many changes to URDF, calibrate kinect, re-arrange arm, etc

File: maxwell/maxwell_defs/urdf/arm.urdf.xacro (robot description, xacro)
@@ -2,9 +2,16 @@
 <robot>
   <macro name="maxwell_arm" params="name parent *origin">
+    <!-- Arm Link -->
+    <joint name="${name}_base_joint" type="fixed">
+      <insert_block name="origin" />
+      <parent link="${parent}_link"/>
+      <child link="${name}_link"/>
+    </joint>
+    <link name="${name}_link"/>
     <!-- Shoulder pan -->
     <joint name="${name}_shoulder_pan_joint" type="revolute">
       <axis xyz="0 0 1" />
-      <insert_block name="origin" />
-      <parent link="${parent}_link"/>
+      <origin xyz="0 0 0" rpy="0 0 0" />
+      <parent link="${name}_link"/>
       <child link="${name}_shoulder_pan_link"/>
       <limit lower="-1.57"  upper="1.57" effort="5.0" velocity="5" />
@@ -28,6 +35,7 @@
     <joint name="${name}_shoulder_lift_joint" type="revolute">
       <axis xyz="0 1 0"/>
+      <origin xyz="0 0 0" rpy="0 -1.57 0" />
+      <!--<origin xyz="0 0 0.0759" rpy="0 -1.57 0" />-->
       <limit lower="-0.2" upper="2.617" effort="5.0" velocity="5" />
-      <origin xyz="0 0 0.0759" rpy="0 -1.57 0" />
       <parent link="${name}_shoulder_pan_link"/>
       <child link="${name}_shoulder_lift_link"/>

File: maxwell/maxwell_defs/urdf/base.urdf.xacro (robot description, xacro)
@@ -2,4 +2,5 @@
 <robot>
   <include filename="$(find maxwell_defs)/urdf/sensors/hokuyo_urg_laser.urdf.xacro" />
+  <property name="ground_clearance" value="0.0238" />
   <!-- simplified box collision geometry for base -->
   <property name="wheels_offset_x" value="0.12065" />
@@ -37,5 +38,5 @@
     <link name="${name}_link">
       <visual>
-        <origin xyz="0 0 0.0238" rpy="0 0 0" />
+        <origin xyz="0 0 ${ground_clearance}" rpy="0 0 0" />
         <geometry>
           <mesh filename="package://maxwell_defs/meshes/base.stl"  />

File: maxwell/maxwell_defs/urdf/gripper.urdf.xacro (robot description, xacro)
@@ -4,5 +4,5 @@
     <joint name="${prefix}_finger_joint" type="revolute">
       <axis xyz="0 0 1" />
-      <origin xyz="-0.012 ${reflect*0.033/2} 0" rpy="0 0 0" />
+      <origin xyz="-0.062 ${reflect*0.033/2} 0" rpy="0 0 0" />
       <limit lower="-1.57"  upper="1.57" effort="5.0" velocity="5" />
       <parent link="${parent}_link"/>

File: maxwell/maxwell_defs/urdf/head.urdf.xacro (robot description, xacro)
@@ -1,34 +1,13 @@
 <?xml version="1.0"?>
 <robot>
+  <!-- origin is center of head tilt rotation -->
   <macro name="maxwell_head" params="name parent *origin">
-    <!-- Head base -->
-    <joint name="${name}_base_joint" type="fixed">
-      <axis xyz="0 1 0" />
-      <insert_block name="origin" />
-      <parent link="${parent}_link"/>
-      <child link="${name}_base_link"/>
-    </joint>
-    <link name="${name}_base_link">
-      <visual>
-        <origin xyz="${-0.0635/4} 0 ${0.0381/2}" rpy="0 0 0" />
-        <geometry>
-          <box size=".0635 .0381 .0381"/>
-        </geometry>
-        <material name="Black" />
-      </visual>
-      <collision>
-        <origin xyz="${-0.0635/4} 0 ${0.0381/2}" rpy="0 0 0" />
-        <geometry>
-          <box size=".0635 .0381 .0381"/>
-        </geometry>
-      </collision>
-    </link>
     <!-- Head pan -->
     <joint name="${name}_pan_joint" type="revolute">
       <axis xyz="0 0 1" />
-      <limit lower="-2.617" upper="2.617" effort="5.0" velocity="5" />
-      <origin xyz="0 0 0.040" rpy="0 0 0" />
-      <parent link="${name}_base_link"/>
+      <insert_block name="origin" />
+      <parent link="${parent}_link"/>
       <child link="${name}_pan_link"/>
+      <limit lower="-2.617" upper="2.617" effort="1" velocity="1" />
     </joint>
     <link name="${name}_pan_link">
@@ -36,5 +15,5 @@
         <origin xyz="0 0 ${0.0635/2}" rpy="0 0 0 " />
         <geometry>
-          <box size=".0381 .0381 .0635"/>
+          <box size="${ax12_depth} ${ax12_width} ${ax12_height+0.00635}"/>
         </geometry>
         <material name="Black" />
@@ -43,5 +22,5 @@
         <origin xyz="0 0 ${0.0635/2}" rpy="0 0 0 " />
         <geometry>
-          <box size=".0381 .0381 .0635"/>
+          <box size="${ax12_depth} ${ax12_width} ${ax12_height+0.00635}"/>
         </geometry>
       </collision>
@@ -51,5 +30,5 @@
       <axis xyz="0 1 0" />
       <limit lower="-1.57" upper="1.57" effort="5.0" velocity="5" />
-      <origin xyz="0 0 0.045" rpy="0 0 0" />
+      <origin xyz="0 0 0" rpy="0 0 0" />
       <parent link="${name}_pan_link"/>
       <child link="${name}_tilt_link"/>
@@ -72,5 +51,5 @@
     <!-- Head sensor frame -->
     <joint name="${name}_sensor_frame_joint" type="fixed">
-      <origin xyz="0 0 0.05" rpy="0 0 0" />
+      <origin xyz="${calib_cam_x} ${calib_cam_y} ${calib_cam_z}" rpy="${calib_cam_rr} ${calib_cam_rp} ${calib_cam_ry}" />
       <parent link="${name}_tilt_link"/>
       <child link="${name}_sensor_frame"/>
@@ -78,5 +57,5 @@
     <link name="${name}_sensor_frame">
       <visual>
-        <origin xyz="-0.0254 0 0" rpy="0 0 -1.57" />
+        <origin xyz="${-calib_cam_x-0.0254} 0 0" rpy="0 0 -1.57" />
         <geometry>
           <mesh filename="package://maxwell_defs/meshes/kinect.stl" />
@@ -84,6 +63,5 @@
         <material name="Black" />
       </visual>
-      <!-- TODO: add collision -->
-    </link>
+    </link> <!-- comment this link out for calibration -->
   </macro>
 </robot>

File: maxwell/maxwell_defs/urdf/maxwell.urdf.xacro (robot description, xacro)
@@ -1,7 +1,22 @@
 <?xml version="1.0"?>
 <robot name="maxwell" >
+  <!-- interactive calibration output:
+        [ INFO] [1310855144.314114846]: -0.0184416, -7.34934e-11, 0.07469, 0.0120684, 0.00708517, -8.5516e-05, 0.999902
+        [ INFO] [1310858627.105328692]: 0.00927514, 0.00208817, 0.0877625, 0.0240435, 0.0424938, 0.00594516, 0.998789
+        [ INFO] [1310858627.105465208]: 0.00927514, 0.00208817, 0.0877625, 0.048728, 0.0847001, 0.0139699
+  -->
+  <property name="calib_cam_x" value="0.00927514" />
+  <property name="calib_cam_y" value="0.00208817" />
+  <property name="calib_cam_z" value="0.0877625" />
+  <property name="calib_cam_rr" value="0.048728" />
+  <property name="calib_cam_rp" value="0.0847001" />
+  <property name="calib_cam_ry" value="0.0139699" />
+  <property name="ax12_height" value="0.04762" />
+  <property name="ax12_width" value="0.0381" />
+  <property name="ax12_depth" value="0.0318" />
+  <property name="ax12_center" value="0.0385" />
   <!-- height properties -->
-  <property name="torso_height" value="0.6" />
-  <property name="column_height" value="1.17475" />
+  <property name="arm_height" value="0.885825" /> <!-- height to shoulder lift rotation -->
+  <property name="column_height" value="1.397" /> <!-- height to neck tilt rotation -->
   <!-- The following included files set up definitions of parts of the robot body -->
   <include filename="$(find maxwell_defs)/urdf/base.urdf.xacro" />
@@ -15,17 +30,17 @@
   <!-- Add Torso Upright -->
   <maxwell_torso name="torso" parent="base">
-    <origin xyz="-0.00635 0 ${0.1397+torso_height}"/>
+    <origin xyz="-0.00635 0 ${arm_height}"/>
   </maxwell_torso>
   <!-- Arm -->
   <maxwell_arm name="arm" parent="torso">
-    <origin xyz="0.0608 0 0.0"/>
+    <origin xyz="0.0608 0 0"/>
   </maxwell_arm>
   <!-- Gripper -->
   <maxwell_gripper name="gripper" parent="arm_wrist_roll">
-    <origin xyz="0.100 0 0" />
+    <origin xyz="0.150 0 0" />
   </maxwell_gripper>
   <!-- Kinect head -->
-  <maxwell_head name="head" parent="torso">
-    <origin xyz="0.0157 0 ${column_height-torso_height}"/>
+  <maxwell_head name="head" parent="base">
+    <origin xyz="0.0157 0 ${column_height}"/>
   </maxwell_head>
 </robot>

File: maxwell/maxwell_defs/urdf/torso.urdf.xacro (robot description, xacro)
@@ -10,5 +10,5 @@
     <link name="${name}_link">
       <visual>
-        <origin xyz="0 0 ${column_height/2-torso_height}" rpy="0 0 0 " />
+        <origin xyz="0 0 ${column_height/2-arm_height}" rpy="0 0 0 " />
         <geometry>
           <box size="0.0254 0.0254 ${column_height}"/>
@@ -17,5 +17,5 @@
       </visual>
       <collision>
-        <origin xyz="0 0 ${column_height/2-torso_height}" rpy="0 0 0 " />
+        <origin xyz="0 0 ${column_height/2-arm_height}" rpy="0 0 0 " />
         <geometry>
           <box size="0.0254 0.0254 ${column_height}"/>
