Commit message: (maxwell_defs) upgrade meshes of arm, cleanup ax12 xacro files

File: maxwell/maxwell_defs/urdf/arm.urdf.xacro (robot description, xacro)
@@ -1,4 +1,28 @@
 <?xml version="1.0"?>
 <robot>
+  <!-- standoffs -->
+  <macro name="standoffs" params="name parent *origin">
+    <joint name="${name}_joint" type="fixed">
+      <insert_block name="origin" />
+      <parent link="${parent}"/>
+      <child link="${name}_link" />
+    </joint>
+    <link name="${name}_link">
+      <visual>
+        <origin xyz="${0.0381/2} 0 0" rpy="0 0 0" />
+        <geometry>
+          <box size="0.0381 0.037 0.030"/>
+        </geometry>
+        <material name="Black"/>
+      </visual>
+      <collision>
+        <origin xyz="${0.0381/2} 0 0" rpy="0 0 0" />
+        <geometry>
+          <box size="0.0381 0.037 0.030"/>
+        </geometry>
+      </collision>
+    </link>
+  </macro>
+  <!-- the actual arm -->
   <macro name="maxwell_arm" params="name parent *origin">
     <!-- Arm Link -->
@@ -10,102 +34,44 @@
     <link name="${name}_link"/>
     <!-- Shoulder pan -->
-    <joint name="${name}_shoulder_pan_joint" type="revolute">
-      <axis xyz="0 0 1" />
-      <origin xyz="0 0 0" rpy="0 0 0" />
-      <parent link="${name}_link"/>
-      <child link="${name}_shoulder_pan_link"/>
-      <limit lower="-1.57"  upper="1.57" effort="5.0" velocity="5" />
-    </joint>
-    <link name="${name}_shoulder_pan_link">
-      <visual name="${name}_shoulder_pan_visual">
-        <origin xyz="${-0.065/2+0.0127} 0 0.040" rpy="0 0 0" />
-        <geometry name="${name}_shoulder_pan_visual_geom">
-          <box size="0.065 0.057 0.120"/>
-        </geometry>
-        <material name="Black" />
-      </visual>
-      <collision>
-        <origin xyz="${-0.065/2+0.0127} 0 0.040" rpy="0 0 0" />
-        <geometry>
-          <box size="0.065 0.057 0.120"/>
-        </geometry>
-      </collision>
-    </link>
+    <dynamixel_rx64_pan parent="${name}_link" name="${name}_shoulder_pan_servo" color="Black">
+      <origin xyz="0 0 0" rpy="0 0 0"/>
+    </dynamixel_rx64_pan>
+    <rx64_side_revolute parent="${name}_shoulder_pan_servo_link" name="${name}_shoulder_pan" llimit="-1.57" ulimit="1.57" color="Grey">
+      <origin xyz="0 0 0.0235" rpy="0 -1.57 0"/>
+    </rx64_side_revolute>
     <!-- Shoulder lift -->
-    <joint name="${name}_shoulder_lift_joint" type="revolute">
-      <axis xyz="0 1 0"/>
-      <origin xyz="0 0 0" rpy="0 -1.57 0" />
-      <!--<origin xyz="0 0 0.0759" rpy="0 -1.57 0" />-->
-      <limit lower="-0.2" upper="2.617" effort="5.0" velocity="5" />
-      <parent link="${name}_shoulder_pan_link"/>
-      <child link="${name}_shoulder_lift_link"/>
-    </joint>
-    <link name="${name}_shoulder_lift_link">
-      <visual name="${name}_shoulder_lift_visual">
-        <origin xyz="${0.165/2} 0 0" rpy="0 0 0" />
-        <geometry name="${name}_shoulder_lift_visual_geom">
-          <box size="0.165 0.057 0.040"/>
-        </geometry>
-        <material name="Grey" />
-      </visual>
-      <collision>
-        <origin xyz="${0.165/2} 0 0" rpy="0 0 0" />
-        <geometry>
-          <box size="0.165 0.057 0.040"/>
-        </geometry>
-      </collision>
-    </link>
+    <dynamixel_rx64_tilt parent="${name}_shoulder_pan_link" name="${name}_shoulder_lift_servo" color="Black">
+      <origin xyz="${0.0611-0.013+0.0045} 0 0" rpy="0 0 0"/>
+    </dynamixel_rx64_tilt>
+    <rx64_hinge_hxl parent="${name}_shoulder_lift_servo_link" name="${name}_shoulder_lift" llimit="-0.2" ulimit="2.617" color="Grey">
+      <origin xyz="0 0 0.0" rpy="0 0 0"/>
+    </rx64_hinge_hxl>
+    <standoffs parent="${name}_shoulder_lift_link" name="${name}_shoulder_standoff">
+      <origin xyz="${0.048+0.0235} 0 0.0" rpy="0 0 0"/>
+    </standoffs>
     <!-- Elbow -->
-    <joint name="${name}_elbow_flex_joint" type="revolute">
-      <axis xyz="0 1 0" />
-      <limit lower="-1.57" upper="2.617" effort="5.0" velocity="5" />
-      <origin xyz="0.165 0 0" rpy="0 0 0" />
-      <parent link="${name}_shoulder_lift_link"/>
-      <child link="${name}_elbow_flex_link"/>
-    </joint>
-    <link name="${name}_elbow_flex_link">
-      <visual name="${name}_elbow_flex_visual">
-        <origin xyz="${0.125/2} 0 0" rpy="0 0 0" />
-        <geometry>
-          <!--<mesh filename="package://pr2_defs/meshes/shoulder_yaw.stl" />-->
-          <box size="0.125 0.057 0.040"/>
-        </geometry>
-        <material name="Black" />
-      </visual>
-      <collision>
-        <origin xyz="${0.125/2} 0 0" rpy="0 0 0" />
-        <geometry>
-          <box size="0.125 0.057 0.040"/>
-        </geometry>
-      </collision>
-    </link>
+    <rx64_side_fixed parent="${name}_shoulder_standoff_link" name="${name}_elbow_flex_fixed" color="Grey">
+      <origin xyz="0.0381 0 0" rpy="0 0 0"/>
+    </rx64_side_fixed>
+    <dynamixel_rx64_tilt parent="${name}_elbow_flex_fixed_link" name="${name}_eblow_flex_servo" color="Black">
+      <origin xyz="${0.0611-0.013+0.0045} 0 0" rpy="0 0 0"/>
+    </dynamixel_rx64_tilt>
+    <rx64_hinge_hxl parent="${name}_eblow_flex_servo_link" name="${name}_elbow_flex" llimit="-1.57" ulimit="2.617" color="Grey">
+      <origin xyz="0 0 0.0" rpy="0 0 0"/>
+    </rx64_hinge_hxl>
     <!-- Wrist flex -->
-    <joint name="${name}_wrist_flex_joint" type="revolute">
-      <axis xyz="0 1 0" />
-      <limit lower="-1.57" upper="1.57" effort="5.0" velocity="5" />
-      <origin xyz="0.125 0 0" rpy="0 0 0" />
-      <parent link="${name}_elbow_flex_link"/>
-      <child link="${name}_wrist_flex_link"/>
-    </joint>
-    <link name="${name}_wrist_flex_link">
-      <visual name="${name}_wrist_flex_visual">
-        <origin xyz="${0.030/2} 0 0" rpy="0 0 0" />
-        <geometry name="${name}_wrist_flex_visual_geom">
-          <!--<mesh filename="package://pr2_defs/meshes/wrist_flex.stl" />-->
-          <box size="0.030 0.057 0.040"/>
-        </geometry>
-        <material name="Grey" />
-      </visual>
-      <collision>
-        <origin xyz="${0.030/2} 0 0" rpy="0 0 0" />
-        <geometry>
-          <box size="0.030 0.057 0.040"/>
-        </geometry>
-      </collision>
-    </link>
+    <rx64_side_fixed parent="${name}_elbow_flex_link" name="${name}_wrist_flex_fixed" color="Grey">
+      <origin xyz="${0.048+0.0235} 0 0" rpy="0 0 0"/>
+    </rx64_side_fixed>
+    <dynamixel_rx64_tilt parent="${name}_wrist_flex_fixed_link" name="${name}_wrist_flex_servo" color="Black">
+      <origin xyz="${0.0611-0.013+0.0045} 0 0" rpy="0 0 0"/>
+    </dynamixel_rx64_tilt>
+    <rx64_hinge parent="${name}_wrist_flex_servo_link" name="${name}_wrist_flex" llimit="-1.57" ulimit="1.57" color="Grey">
+      <origin xyz="0 0 0.0" rpy="0 0 0"/>
+    </rx64_hinge>
     <!-- Wrist roll -->
     <joint name="${name}_wrist_roll_joint" type="revolute">
       <axis xyz="1 0 0" />
-      <limit lower="-2.617" upper="2.617" effort="5.0" velocity="5" />
+      <limit effort="30" velocity="1.0" lower="-2.617" upper="2.617"/>
       <origin xyz="0.030 0 0" rpy="0 0 0" />
       <parent link="${name}_wrist_flex_link"/>
@@ -113,16 +79,22 @@
     </joint>
     <link name="${name}_wrist_roll_link">
-      <visual name="${name}_wrist_roll_visual">
-        <origin xyz="0.05 0 0" rpy="0 0 0" />
-        <geometry name="${name}_wrist_roll_visual_geom">
-          <!--<mesh filename="package://pr2_defs/meshes/wrist_roll.stl" />-->
-          <box size="0.100 0.065 0.050"/>
+      <inertial>
+        <mass value="0.00001" />
+        <origin xyz="0 0 0" />
+        <inertia ixx="1.0" ixy="0.0" ixz="0.0"
+          iyy="1.0" iyz="0.0"
+          izz="1.0" />
+      </inertial>
+      <visual>
+        <origin xyz="${0.0425/2} 0 0" rpy="0 0 1.57" />
+        <geometry>
+          <mesh filename="package://maxwell_defs/meshes/ax12.stl" scale="0.001 0.001 0.001"/>
         </geometry>
-        <material name="Black" />
+        <material name="Black"/>
       </visual>
       <collision>
-        <origin xyz="0.05 0 0" rpy="0 0 0" />
+        <origin xyz="-0.01241 0.0 0.0" rpy="0 0 0" />
         <geometry>
-          <box size="0.100 0.065 0.050"/>
+          <box size="0.04762 0.028 0.038"/>
         </geometry>
       </collision>

File: maxwell/maxwell_defs/urdf/head.urdf.xacro (robot description, xacro)
@@ -1,84 +1,26 @@
 <?xml version="1.0"?>
 <robot>
-  <property name="M_PI" value="3.14159"/>
-  <property name="AX12_WIDTH" value="0.038"/>
-  <property name="AX12_HEIGHT" value="0.0385"/>
-  <property name="F10_HEIGHT" value="0.004"/>
-  <include filename="$(find maxwell_defs)/urdf/hardware/bioloid_ax12.xacro" />
-  <include filename="$(find maxwell_defs)/urdf/hardware/bioloid_F2_revolute.xacro" />
-  <include filename="$(find maxwell_defs)/urdf/hardware/bioloid_F3_revolute.xacro" />
-  <include filename="$(find maxwell_defs)/urdf/hardware/bioloid_F3_fixed.xacro" />
   <!-- origin is center of head tilt rotation -->
   <macro name="maxwell_head" params="name parent *origin">
     <!-- Head pan -->
-    <joint name="${name}_pan_servo_joint" type="fixed">
+    <dynamixel_ax12_pan parent="${parent}" name="${name}_pan_servo" color="Black">
       <insert_block name="origin" />
-      <parent link="${parent}"/>
-      <child link="${name}_pan_servo_link" />
-    </joint>
-    <link name="${name}_pan_servo_link">
-      <inertial>
-        <mass value="0.00001" />
-        <origin xyz="0 0 0" />
-        <inertia ixx="1.0" ixy="0.0" ixz="0.0"
-          iyy="1.0" iyz="0.0"
-          izz="1.0" />
-      </inertial>
-      <visual>
-        <origin xyz="0 0 0" rpy="1.57 0 1.57" />
-        <geometry>
-          <mesh filename="package://maxwell_defs/meshes/ax12_box.stl" scale="0.001 0.001 0.001"/>
-        </geometry>
-        <material name="Black"/>
-      </visual>
-      <collision>
-        <origin xyz="-0.01241 0.0 0.0" rpy="1.57 0 1.57" />
-        <geometry>
-          <box size="0.025 0.038 0.04762"/>
-        </geometry>
-      </collision>
-    </link>
-    <joint name="${name}_pan_joint" type="revolute">
-      <origin xyz="0 0 ${AX12_WIDTH/2}"/>
-      <axis xyz="0 0 1"/>
-      <limit effort="30" velocity="1.0" lower="-2.61799388" upper="2.61799388" />
-      <parent link="${name}_pan_servo_link"/>
-      <child link="${name}_pan_link" />
-    </joint>
-    <link name="${name}_pan_link">
-      <inertial>
-        <mass value="0.00001" />
-        <origin xyz="0 0 0" />
-        <inertia ixx="1.0" ixy="0.0" ixz="0.0"
-          iyy="1.0" iyz="0.0"
-          izz="1.0" />
-      </inertial>
-      <visual>
-        <origin xyz=" 0 0 0 " rpy="3.14 0 0" />
-        <geometry>
-          <mesh filename="package://maxwell_defs/meshes/F3.stl" scale="0.001 0.001 0.001"/>
-        </geometry>
-        <material name="Black"/>
-      </visual>
-      <collision>
-        <origin xyz="0.0 0.0 0.0045" rpy="0 0 0" />
-        <geometry>
-          <box size="0.025 0.038 0.009"/>
-        </geometry>
-      </collision>
-    </link>
-    <bioloid_F3_fixed parent="${name}_pan_servo_link" name="${name}_tilt_left_side" joint_name="${name}_tilt_left_joint" color="Black">
+    </dynamixel_ax12_pan>
+    <ax12_side_revolute parent="${name}_pan_servo_link" name="${name}_pan" llimit="-2.617" ulimit="2.617" color="Orange">
+      <origin xyz="0 0 ${AX12_WIDTH/2}" rpy="0 0 0"/>
+    </ax12_side_revolute>
+    <ax12_side_fixed parent="${name}_pan_servo_link" name="${name}_tilt_left_side" color="Black">
       <origin xyz="-0.015 ${-AX12_WIDTH/2} 0" rpy="1.57 0 0"/>
-    </bioloid_F3_fixed>
-    <bioloid_F3_fixed parent="${name}_pan_servo_link" name="${name}_tilt_right_side" joint_name="${name}_tilt_right_joint" color="Black">
+    </ax12_side_fixed>
+    <ax12_side_fixed parent="${name}_pan_servo_link" name="${name}_tilt_right_side" color="Black">
       <origin xyz="-0.015 ${AX12_WIDTH/2} 0" rpy="-1.57 0 0"/>
-    </bioloid_F3_fixed>
+    </ax12_side_fixed>
     <!-- Head tilt -->
-    <bioloid_ax12 parent="${name}_pan_link" name="${name}_tilt_servo" color="Black">
+    <dynamixel_ax12_tilt parent="${name}_pan_link" name="${name}_tilt_servo" color="Black">
       <origin xyz="0 0 ${AX12_HEIGHT+F10_HEIGHT-0.001}" rpy="0 0 0"/>
-    </bioloid_ax12>
-    <bioloid_F2_revolute parent="${name}_tilt_servo_link" name="${name}_tilt" joint_name="${name}_tilt_joint" color="Orange">
+    </dynamixel_ax12_tilt>
+    <ax12_hinge_revolute parent="${name}_tilt_servo_link" name="${name}_tilt" color="Orange">
      <origin xyz="0 0 0" rpy="0 0 0"/>
-    </bioloid_F2_revolute>
+    </ax12_hinge_revolute>
     <!-- Head sensor frame -->
     <joint name="${name}_sensor_frame_joint" type="fixed">

File: maxwell/maxwell_defs/urdf/maxwell.urdf.xacro (robot description, xacro)
@@ -16,18 +16,13 @@
   <property name="calib_cam_ry" value="0" />
   -->
-  <property name="ax12_height" value="0.04762" />
-  <property name="ax12_width" value="0.0381" />
-  <property name="ax12_depth" value="0.0318" />
-  <property name="ax12_center" value="0.0385" />
-  <!-- height properties -->
-  <!--<property name="arm_height" value="0.885825" /> height to shoulder lift rotation -->
-   <!--<property name="column_height" value="1.397" /> height to neck tilt rotation -->
-  <property name="arm_height" value="0.5921375" /> <!-- deck to bottom of arm mount TODO: update this -->
+  <property name="arm_height" value="0.6619375 " /> <!-- deck to arm_link -->
   <property name="column_height" value="1.171575" /> <!-- deck to top of 80/20: 46-1/8" -->
+  <include filename="$(find maxwell_defs)/urdf/hardware/ax12.xacro" />
+  <include filename="$(find maxwell_defs)/urdf/hardware/rx64.xacro" />
   <!-- The following included files set up definitions of parts of the robot body -->
   <include filename="$(find maxwell_defs)/urdf/base.urdf.xacro" />
   <include filename="$(find maxwell_defs)/urdf/torso.urdf.xacro" />
   <include filename="$(find maxwell_defs)/urdf/arm.urdf.xacro" />
-  <include filename="$(find maxwell_defs)/urdf/gripper.urdf.xacro" />
+  <!--<include filename="$(find maxwell_defs)/urdf/gripper.urdf.xacro" />-->
   <include filename="$(find maxwell_defs)/urdf/head.urdf.xacro" />
   <include filename="$(find maxwell_defs)/urdf/materials.urdf.xacro" />
@@ -40,10 +35,10 @@
   <!-- Arm -->
   <maxwell_arm name="arm" parent="torso">
-    <origin xyz="0.0608 0 ${arm_height+.15}"/>
+    <origin xyz="0.0608 0 ${arm_height}"/>
   </maxwell_arm>
   <!-- Gripper -->
-  <maxwell_gripper name="gripper" parent="arm_wrist_roll">
+  <!--<maxwell_gripper name="gripper" parent="arm_wrist_roll">
     <origin xyz="0.150 0 0" />
-  </maxwell_gripper>
+  </maxwell_gripper>-->
   <!-- Kinect head -->
   <maxwell_head name="head" parent="torso_link">

Commit message: (maxwell_defs) fix wrist roll collision model

File: maxwell/maxwell_defs/urdf/arm.urdf.xacro (robot description, xacro)
@@ -94,7 +94,7 @@
       </visual>
       <collision>
-        <origin xyz="-0.01241 0.0 0.0" rpy="0 0 0" />
+        <origin xyz="${0.0425/2} 0.0 -0.01241 " rpy="0 0 0" />
         <geometry>
-          <box size="0.04762 0.028 0.038"/>
+          <box size="0.038 0.028 0.04762"/>
         </geometry>
       </collision>
