Commit message: (maxwell_defs) finish rework of URDF

File: maxwell/maxwell_defs/urdf/arm.urdf.xacro (robot description, xacro)
@@ -24,4 +24,27 @@
     </link>
   </macro>
+  <!-- cosmetics -->
+  <macro name="arm_mount" params="name parent *origin">
+    <joint name="${name}_joint" type="fixed">
+      <insert_block name="origin" />
+      <parent link="${parent}"/>
+      <child link="${name}_link" />
+    </joint>
+    <link name="${name}_link">
+      <visual>
+        <origin xyz="0 0 0" rpy="1.57 3.14 0" />
+        <geometry>
+          <mesh filename="package://maxwell_defs/meshes/arm_mount.stl" scale="1 1 1"/>
+        </geometry>
+        <material name="Black"/>
+      </visual>
+      <collision>
+        <origin xyz="0.03055 ${-0.0047625/2} 0" rpy="0 0 0" />
+        <geometry>
+          <box size="0.0865 0.0047625 0.038"/>
+        </geometry>
+      </collision>
+    </link>
+  </macro>
   <!-- the actual arm -->
   <macro name="maxwell_arm" params="name parent *origin">
@@ -33,4 +56,10 @@
     </joint>
     <link name="${name}_link"/>
+    <arm_mount name="${name}_left_mount" parent="${name}_link">
+      <origin xyz="-0.0611 0.0254 0" rpy="0 0 0"/>
+    </arm_mount>
+    <arm_mount name="${name}_right_mount" parent="${name}_link">
+      <origin xyz="-0.0611 ${-0.0254+0.0047625} 0" rpy="0 0 0"/>
+    </arm_mount>
     <!-- Shoulder pan -->
     <dynamixel_rx64_pan parent="${name}_link" name="${name}_shoulder_pan_servo" color="Black">
@@ -74,5 +103,5 @@
       <axis xyz="1 0 0" />
       <limit effort="30" velocity="1.0" lower="-2.617" upper="2.617"/>
-      <origin xyz="0.030 0 0" rpy="0 0 0" />
+      <origin xyz="0.031 0 0" rpy="0 0 0" />
       <parent link="${name}_wrist_flex_link"/>
       <child link="${name}_wrist_roll_link"/>
@@ -87,5 +116,5 @@
       </inertial>
       <visual>
-        <origin xyz="${0.0425/2} 0 0" rpy="0 0 1.57" />
+        <origin xyz="${0.0381/2} 0 0" rpy="0 0 1.57" />
         <geometry>
           <mesh filename="package://maxwell_defs/meshes/ax12.stl" scale="0.001 0.001 0.001"/>
@@ -94,7 +123,7 @@
       </visual>
       <collision>
-        <origin xyz="${0.0425/2} 0.0 -0.01241 " rpy="0 0 0" />
+        <origin xyz="${0.0381/2} 0.0 -0.01241 " rpy="0 0 0" />
         <geometry>
-          <box size="0.038 0.028 0.04762"/>
+          <box size="0.0381 0.028 0.04762"/>
         </geometry>
       </collision>

File: maxwell/maxwell_defs/urdf/gripper.urdf.xacro (robot description, xacro)
@@ -1,39 +1,55 @@
 <?xml version="1.0"?>
 <robot>
-  <macro name="gripper_finger" params="prefix parent reflect">
-    <joint name="${prefix}_finger_joint" type="revolute">
-      <axis xyz="0 0 1" />
-      <origin xyz="-0.062 ${reflect*0.033/2} 0" rpy="0 0 0" />
-      <limit lower="-1.57"  upper="1.57" effort="5.0" velocity="5" />
-      <parent link="${parent}_link"/>
-      <child link="${prefix}_finger_link"/>
-    </joint>
-    <link name="${prefix}_finger_link">
-      <visual name="${prefix}_finger_visual">
-        <origin xyz="0 0 0" rpy="0 0 0" />
-        <geometry name="${prefix}_finger_visual_geom">
-          <box size="0.125 0.01 0.03"/>
-        </geometry>
-        <material name="Orange" />
-      </visual>
-      <collision>
-        <origin xyz="0 0 0" rpy="0 0 0" />
-        <geometry>
-          <box size="0.125 0.01 0.03"/>
-        </geometry>
-      </collision>
-    </link>
-  </macro>
   <macro name="maxwell_gripper" params="name parent *origin">
-    <!-- Base of Gripper Pad -->
+    <ax12_F6_fixed parent="${parent}_link" name="${name}_F6_1" color="Black">
+      <origin xyz="${0.0381/2} 0.017 -0.014" rpy="0 0 0"/>
+    </ax12_F6_fixed>
+    <ax12_F6_fixed parent="${name}_F6_1_link" name="${name}_F6_2" color="Black">
+      <origin xyz="0.008 0.004 0" rpy="3.14 3.14 0"/>
+    </ax12_F6_fixed>
+    <ax12_F6_fixed parent="${parent}_link" name="${name}_F6_3" color="Black">
+      <origin xyz="${0.0381/2} -0.017 -0.014" rpy="3.14 0 0"/>
+    </ax12_F6_fixed>
+    <ax12_F6_fixed parent="${name}_F6_3_link" name="${name}_F6_4" color="Black">
+      <origin xyz="0.008 0.004 0" rpy="0 0 3.14"/>
+    </ax12_F6_fixed>
+    <ax12_side_fixed parent="${name}_F6_2_link" name="left_${name}_mount" color="Black">
+      <origin xyz="-0.018 0.005 0" rpy="1.57 0 1.57"/>
+    </ax12_side_fixed>
+    <ax12_side_fixed parent="${name}_F6_4_link" name="right_${name}_mount" color="Black">
+      <origin xyz="-0.018 0.005 0" rpy="1.57 0 1.57"/>
+    </ax12_side_fixed>
+    <dynamixel_ax12_pan parent="left_${name}_mount_link" name="left_${name}_servo" color="Black">
+      <origin xyz="0 0 -0.042" rpy="-1.57 1.57 0"/>
+    </dynamixel_ax12_pan>
+    <dynamixel_ax12_pan parent="right_${name}_mount_link" name="right_${name}_servo" color="Black">
+      <origin xyz="0 0 -0.042" rpy="1.57 1.57 0"/>
+    </dynamixel_ax12_pan>
+    <ax12_F1_revolute parent="left_${name}_servo_link" name="l_${name}" llimit="-1.57" ulimit="1.57" color="Orange">
+      <origin xyz="0 0 0" rpy="3.14 0 1.57"/>
+    </ax12_F1_revolute>
+    <ax12_F1_revolute parent="right_${name}_servo_link" name="r_${name}" llimit="-1.57" ulimit="1.57" color="Orange">
+      <origin xyz="0 0 0" rpy="0 0 -1.57"/>
+    </ax12_F1_revolute>
+    <ax12_F9_fixed parent="l_${name}_link" name="left_${name}_F9" color="Black">
+      <origin xyz="0.0155 0.038 0" rpy="0 3.14 0"/>
+    </ax12_F9_fixed>
+    <ax12_F9_fixed parent="r_${name}_link" name="right_${name}_F9" color="Black">
+      <origin xyz="0.0155 0.038 0" rpy="0 3.14 0"/>
+    </ax12_F9_fixed>
+    <ax12_F11_fixed parent="left_${name}_F9_link" name="left_${name}_finger" color="Grey">
+      <origin xyz="0 -0.013 0 " rpy="0 0 0"/>
+    </ax12_F11_fixed>
+    <ax12_F11_fixed parent="right_${name}_F9_link" name="right_${name}_finger" color="Grey">
+      <origin xyz="0 -0.013 0" rpy="0 0 0"/>
+    </ax12_F11_fixed>
+    <!-- Gripper Joint for Grasping -->
     <joint name="${name}_joint" type="fixed">
       <axis xyz="0 0 1" />
-      <insert_block name="origin" />
+      <origin xyz="0.16 0 -0.012" rpy="0 0 0"/>
       <parent link="${parent}_link"/>
       <child link="${name}_link"/>
     </joint>
     <link name="${name}_link"/>
-    <gripper_finger prefix="l" parent="gripper" reflect="1"/>
-    <gripper_finger prefix="r" parent="gripper" reflect="-1" />
   </macro>
 </robot>

File: maxwell/maxwell_defs/urdf/hardware/ax12.xacro (robot description, xacro)
@@ -1,12 +1,6 @@
 <?xml version="1.0"?>
 <robot>
-  <property name="M_PI" value="3.14159"/>
   <property name="AX12_WIDTH" value="0.038"/>
   <property name="AX12_HEIGHT" value="0.0385"/>
-  <property name="F10_HEIGHT" value="0.004"/>
-  <property name="ax12_height" value="0.04762" />
-  <property name="ax12_width" value="0.0381" />
-  <property name="ax12_depth" value="0.0318" />
-  <property name="ax12_center" value="0.0385" />
   <macro name="dynamixel_ax12_pan" params="parent name color *origin" >
     <joint name="${name}_joint" type="fixed">
@@ -158,3 +152,121 @@
     </link>
   </macro>
+  <macro name="ax12_F1_revolute" params="name parent color llimit ulimit *origin">
+    <joint name="${name}_joint" type="revolute">
+      <insert_block name="origin" />
+       <axis xyz="0 0 1"/>
+      <limit effort="30" velocity="1.0" lower="${llimit}" upper="${ulimit}" />
+      <parent link="${parent}"/>
+      <child link="${name}_link" />
+    </joint>
+    <link name="${name}_link">
+      <inertial>
+        <mass value="0.00001" />
+        <origin xyz="0 0 0" />
+        <inertia ixx="1.0" ixy="0.0" ixz="0.0"
+          iyy="1.0" iyz="0.0"
+          izz="1.0" />
+      </inertial>
+      <visual>
+        <origin xyz=" 0 0 0 " rpy="3.14 0 0" />
+        <geometry>
+          <mesh filename="package://maxwell_defs/meshes/F1.stl" scale="1 1 1"/>
+        </geometry>
+        <material name="${color}"/>
+      </visual>
+      <collision>
+        <origin xyz="0.01 0.008 0.0" rpy="0 0 .8" />
+        <geometry>
+          <box size="0.04 0.028 0.046"/>
+        </geometry>
+      </collision>
+    </link>
+  </macro>
+  <macro name="ax12_F6_fixed" params="name parent color *origin">
+    <joint name="${name}_joint" type="fixed">
+      <insert_block name="origin" />
+      <parent link="${parent}"/>
+      <child link="${name}_link" />
+    </joint>
+    <link name="${name}_link">
+      <inertial>
+        <mass value="0.00001" />
+        <origin xyz="0 0 0" />
+        <inertia ixx="1.0" ixy="0.0" ixz="0.0"
+          iyy="1.0" iyz="0.0"
+          izz="1.0" />
+      </inertial>
+      <visual>
+        <origin xyz=" 0 0 0 " rpy="3.14 0 0" />
+        <geometry>
+          <mesh filename="package://maxwell_defs/meshes/F6.stl" scale="1 1 1"/>
+        </geometry>
+        <material name="${color}"/>
+      </visual>
+      <collision>
+        <origin xyz="0.001 0.0 0.0" rpy="0 0 0" />
+        <geometry>
+          <box size="0.04 0.005 0.024"/>
+        </geometry>
+      </collision>
+    </link>
+  </macro>
+  <macro name="ax12_F9_fixed" params="name parent color *origin">
+    <joint name="${name}_joint" type="fixed">
+      <insert_block name="origin" />
+      <parent link="${parent}"/>
+      <child link="${name}_link" />
+    </joint>
+    <link name="${name}_link">
+      <inertial>
+        <mass value="0.00001" />
+        <origin xyz="0 0 0" />
+        <inertia ixx="1.0" ixy="0.0" ixz="0.0"
+          iyy="1.0" iyz="0.0"
+          izz="1.0" />
+      </inertial>
+      <visual>
+        <origin xyz="0 0 0" rpy="0 0 0" />
+        <geometry>
+          <mesh filename="package://maxwell_defs/meshes/F9.stl" scale="1 1 1"/>
+        </geometry>
+        <material name="${color}"/>
+      </visual>
+      <collision>
+        <origin xyz="-0.008 0.0 0.0" rpy="0 0 0" />
+        <geometry>
+          <box size="0.008 0.03 0.024"/>
+        </geometry>
+      </collision>
+    </link>
+  </macro>
+  <macro name="ax12_F11_fixed" params="name parent color *origin">
+    <joint name="${name}_joint" type="fixed">
+      <insert_block name="origin" />
+      <parent link="${parent}"/>
+      <child link="${name}_link" />
+    </joint>
+    <link name="${name}_link">
+      <inertial>
+        <mass value="0.00001" />
+        <origin xyz="0 0 0" />
+        <inertia ixx="1.0" ixy="0.0" ixz="0.0"
+          iyy="1.0" iyz="0.0"
+          izz="1.0" />
+      </inertial>
+      <visual>
+        <origin xyz="0 0 0" rpy="0 0 0" />
+        <geometry>
+          <mesh filename="package://maxwell_defs/meshes/F11.stl" scale="1 1 1"/>
+        </geometry>
+        <material name="${color}"/>
+      </visual>
+      <collision>
+        <origin xyz="-0.008 0.025 0.0" rpy="0 0 0" />
+        <geometry>
+          <box size="0.009 0.06 0.028"/>
+        </geometry>
+      </collision>
+    </link>
+  </macro>
 </robot>

File: maxwell/maxwell_defs/urdf/head.urdf.xacro (robot description, xacro)
@@ -18,5 +18,5 @@
     <!-- Head tilt -->
     <dynamixel_ax12_tilt parent="${name}_pan_link" name="${name}_tilt_servo" color="Black">
-      <origin xyz="0 0 ${AX12_HEIGHT+F10_HEIGHT-0.001}" rpy="0 0 0"/>
+      <origin xyz="0 0 ${AX12_HEIGHT+0.003}" rpy="0 0 0"/>
     </dynamixel_ax12_tilt>
     <ax12_hinge_revolute parent="${name}_tilt_servo_link" name="${name}_tilt" color="Orange">
@@ -37,4 +37,10 @@
         <material name="Black" />
       </visual>
+      <collision>
+        <origin xyz="0 0 0" rpy="0 0 0" />
+        <geometry>
+          <box size="0.064 0.28 0.04"/>
+        </geometry>
+      </collision>
     </link>
     <!-- Openni Link -->

File: maxwell/maxwell_defs/urdf/maxwell.urdf.xacro (robot description, xacro)
@@ -4,16 +4,7 @@
   <property name='calib_cam_y' value='0.0060704' />
   <property name='calib_cam_z' value='-0.0306572' />
-  <!--<property name='calib_cam_z' value='0.0118428' />-->
   <property name='calib_cam_rr' value='-0.024976' />
   <property name='calib_cam_rp' value='-0.0119664' />
   <property name='calib_cam_ry' value='0.0228755' />
-  <!--
-  <property name="calib_cam_x" value="0" />
-  <property name="calib_cam_y" value="0" />
-  <property name="calib_cam_z" value="0" />
-  <property name="calib_cam_rr" value="0" />
-  <property name="calib_cam_rp" value="0" />
-  <property name="calib_cam_ry" value="0" />
-  -->
   <property name="arm_height" value="0.6619375 " /> <!-- deck to arm_link -->
   <property name="column_height" value="1.171575" /> <!-- deck to top of 80/20: 46-1/8" -->
@@ -24,5 +15,5 @@
   <include filename="$(find maxwell_defs)/urdf/torso.urdf.xacro" />
   <include filename="$(find maxwell_defs)/urdf/arm.urdf.xacro" />
-  <!--<include filename="$(find maxwell_defs)/urdf/gripper.urdf.xacro" />-->
+  <include filename="$(find maxwell_defs)/urdf/gripper.urdf.xacro" />
   <include filename="$(find maxwell_defs)/urdf/head.urdf.xacro" />
   <include filename="$(find maxwell_defs)/urdf/materials.urdf.xacro" />
@@ -35,14 +26,12 @@
   <!-- Arm -->
   <maxwell_arm name="arm" parent="torso">
-    <origin xyz="0.0608 0 ${arm_height}"/>
+    <origin xyz="0.0611 0 ${arm_height}"/>
   </maxwell_arm>
   <!-- Gripper -->
-  <!--<maxwell_gripper name="gripper" parent="arm_wrist_roll">
-    <origin xyz="0.150 0 0" />
-  </maxwell_gripper>-->
+  <maxwell_gripper name="gripper" parent="arm_wrist_roll">
+    <origin xyz="0 0 0" />
+  </maxwell_gripper>
   <!-- Kinect head -->
   <maxwell_head name="head" parent="torso_link">
-    <!--<origin xyz="0.0157 0 ${column_height}"/>-->
-    <!--<origin xyz="${0.0157+0.05715/2} -0.005 ${column_height+0.0460375}"/>-->
     <origin xyz="0 0 ${column_height+0.0270375}"/>
   </maxwell_head>

File: maxwell/maxwell_defs/urdf/sensors/hokuyo_urg_laser.urdf.xacro (robot description, xacro)
@@ -14,5 +14,5 @@
         <inertia ixx="0.0001" ixy="0" ixz="0" iyy="0.000001" iyz="0" izz="0.0001" />
       </inertial>
-      <visual>
+      <!--<visual>
         <origin xyz="0 0 -0.022" rpy="0 0 0" />
         <geometry>
@@ -20,5 +20,5 @@
         </geometry>
         <material name="Red" />
-      </visual>
+      </visual>-->
       <collision>
         <origin xyz="0 0 -0.022" rpy="0 0 0" />
