Commit message: (maxwell_defs) add joint velocity limits, head_mount stl

File: maxwell/maxwell_defs/urdf/arm.urdf.xacro (robot description, xacro)
@@ -66,5 +66,5 @@
       <origin xyz="0 0 0" rpy="0 0 0"/>
     </dynamixel_rx64_pan>
-    <rx64_side_revolute parent="${name}_shoulder_pan_servo_link" name="${name}_shoulder_pan" llimit="-1.57" ulimit="1.57" color="Grey">
+    <rx64_side_revolute parent="${name}_shoulder_pan_servo_link" name="${name}_shoulder_pan" llimit="-1.57" ulimit="1.57" vlimit="0.524" color="Grey">
       <origin xyz="0 0 0.0235" rpy="0 -1.57 0"/>
     </rx64_side_revolute>
@@ -73,5 +73,5 @@
       <origin xyz="${0.0611-0.013+0.0045} 0 0" rpy="0 0 0"/>
     </dynamixel_rx64_tilt>
-    <rx64_hinge_hxl parent="${name}_shoulder_lift_servo_link" name="${name}_shoulder_lift" llimit="-0.2" ulimit="2.617" color="Grey">
+    <rx64_hinge_hxl parent="${name}_shoulder_lift_servo_link" name="${name}_shoulder_lift" llimit="-0.2" ulimit="2.617" vlimit="0.524" color="Grey">
       <origin xyz="0 0 0.0" rpy="0 0 0"/>
     </rx64_hinge_hxl>
@@ -86,5 +86,5 @@
       <origin xyz="${0.0611-0.013+0.0045} 0 0" rpy="0 0 0"/>
     </dynamixel_rx64_tilt>
-    <rx64_hinge_hxl parent="${name}_elbow_flex_servo_link" name="${name}_elbow_flex" llimit="-1.57" ulimit="2.617" color="Grey">
+    <rx64_hinge_hxl parent="${name}_elbow_flex_servo_link" name="${name}_elbow_flex" llimit="-1.57" ulimit="2.617" vlimit="0.524" color="Grey">
       <origin xyz="0 0 0.0" rpy="0 0 0"/>
     </rx64_hinge_hxl>
@@ -96,5 +96,5 @@
       <origin xyz="${0.0611-0.013+0.0045} 0 0" rpy="0 0 0"/>
     </dynamixel_rx64_tilt>
-    <rx64_hinge parent="${name}_wrist_flex_servo_link" name="${name}_wrist_flex" llimit="-1.57" ulimit="1.57" color="Grey">
+    <rx64_hinge parent="${name}_wrist_flex_servo_link" name="${name}_wrist_flex" llimit="-1.57" ulimit="1.57" vlimit="0.785" color="Grey">
       <origin xyz="0 0 0.0" rpy="0 0 0"/>
     </rx64_hinge>
@@ -102,5 +102,5 @@
     <joint name="${name}_wrist_roll_joint" type="revolute">
       <axis xyz="1 0 0" />
-      <limit effort="30" velocity="1.0" lower="-2.617" upper="2.617"/>
+      <limit effort="30" velocity="0.785" lower="-2.617" upper="2.617"/>
       <origin xyz="0.031 0 0" rpy="0 0 0" />
       <parent link="${name}_wrist_flex_link"/>

File: maxwell/maxwell_defs/urdf/gripper.urdf.xacro (robot description, xacro)
@@ -26,8 +26,8 @@
       <origin xyz="0 0 -0.042" rpy="1.57 1.57 0"/>
     </dynamixel_ax12_pan>
-    <ax12_F1_revolute parent="left_${name}_servo_link" name="l_${name}" llimit="-1.57" ulimit="1.57" color="Orange">
+    <ax12_F1_revolute parent="left_${name}_servo_link" name="l_${name}" llimit="-1.57" ulimit="1.57" vlimit="0.5" color="Orange">
       <origin xyz="0 0 0" rpy="3.14 0 1.57"/>
     </ax12_F1_revolute>
-    <ax12_F1_revolute parent="right_${name}_servo_link" name="r_${name}" llimit="-1.57" ulimit="1.57" color="Orange">
+    <ax12_F1_revolute parent="right_${name}_servo_link" name="r_${name}" llimit="-1.57" ulimit="1.57" vlimit="0.5" color="Orange">
       <origin xyz="0 0 0" rpy="0 0 -1.57"/>
     </ax12_F1_revolute>
@@ -47,5 +47,5 @@
     <joint name="${name}_joint" type="fixed">
       <axis xyz="0 0 1" />
-      <origin xyz="0.16 0 -0.012" rpy="0 0 0"/>
+      <origin xyz="0.16 0 0" rpy="0 0 0"/>
       <parent link="${parent}_link"/>
       <child link="${name}_link"/>

File: maxwell/maxwell_defs/urdf/hardware/ax12.xacro (robot description, xacro)
@@ -61,9 +61,9 @@
     </link>
   </macro>
-  <macro name="ax12_side_revolute" params="name parent llimit ulimit color *origin" >
+  <macro name="ax12_side_revolute" params="name parent llimit ulimit vlimit color *origin" >
     <joint name="${name}_joint" type="revolute">
       <insert_block name="origin" />
       <axis xyz="0 0 1"/>
-      <limit effort="30" velocity="1.0" lower="${llimit}" upper="${ulimit}" />
+      <limit effort="30" velocity="${vlimit}" lower="${llimit}" upper="${ulimit}" />
       <parent link="${parent}"/>
       <child link="${name}_link" />
@@ -121,9 +121,9 @@
     </link>
   </macro>
-  <macro name="ax12_hinge_revolute" params="parent name color *origin">
+  <macro name="ax12_hinge_revolute" params="parent name color llimit ulimit vlimit *origin">
     <joint name="${name}_joint" type="revolute">
       <insert_block name="origin" />
        <axis xyz="0 1 0"/>
-      <limit effort="30" velocity="1.0" lower="-2.61799388" upper="2.61799388" />
+      <limit effort="30" velocity="${vlimit}" lower="${llimit}" upper="${ulimit}" />
       <parent link="${parent}"/>
       <child link="${name}_link" />
@@ -152,9 +152,9 @@
     </link>
   </macro>
-  <macro name="ax12_F1_revolute" params="name parent color llimit ulimit *origin">
+  <macro name="ax12_F1_revolute" params="name parent color llimit ulimit vlimit *origin">
     <joint name="${name}_joint" type="revolute">
       <insert_block name="origin" />
        <axis xyz="0 0 1"/>
-      <limit effort="30" velocity="1.0" lower="${llimit}" upper="${ulimit}" />
+      <limit effort="30" velocity="${vlimit}" lower="${llimit}" upper="${ulimit}" />
       <parent link="${parent}"/>
       <child link="${name}_link" />

File: maxwell/maxwell_defs/urdf/hardware/rx64.xacro (robot description, xacro)
@@ -59,9 +59,9 @@
     </link>
   </macro>
-  <macro name="rx64_side_revolute" params="parent name color llimit ulimit *origin">
+  <macro name="rx64_side_revolute" params="parent name color llimit ulimit vlimit *origin">
     <joint name="${name}_joint" type="revolute">
       <insert_block name="origin" />
        <axis xyz="1 0 0"/>
-      <limit effort="30" velocity="1.0" lower="${llimit}" upper="${ulimit}" />
+      <limit effort="30" velocity="${vlimit}" lower="${llimit}" upper="${ulimit}" />
       <parent link="${parent}"/>
       <child link="${name}_link" />
@@ -119,9 +119,9 @@
     </link>
   </macro>
-  <macro name="rx64_hinge_hxl" params="parent name color llimit ulimit *origin">
+  <macro name="rx64_hinge_hxl" params="parent name color llimit ulimit vlimit *origin">
     <joint name="${name}_joint" type="revolute">
       <insert_block name="origin" />
        <axis xyz="0 1 0"/>
-      <limit effort="30" velocity="1.0" lower="${llimit}" upper="${ulimit}" />
+      <limit effort="30" velocity="${vlimit}" lower="${llimit}" upper="${ulimit}" />
       <parent link="${parent}"/>
       <child link="${name}_link" />
@@ -150,9 +150,9 @@
     </link>
   </macro>
-  <macro name="rx64_hinge" params="parent name color llimit ulimit *origin">
+  <macro name="rx64_hinge" params="parent name color llimit ulimit vlimit *origin">
     <joint name="${name}_joint" type="revolute">
       <insert_block name="origin" />
        <axis xyz="0 1 0"/>
-      <limit effort="30" velocity="1.0" lower="${llimit}" upper="${ulimit}" />
+      <limit effort="30" velocity="${vlimit}" lower="${llimit}" upper="${ulimit}" />
       <parent link="${parent}"/>
       <child link="${name}_link" />

File: maxwell/maxwell_defs/urdf/head.urdf.xacro (robot description, xacro)
@@ -1,11 +1,46 @@
 <?xml version="1.0"?>
 <robot>
+  <!-- cosmetics -->
+  <macro name="head_mount" params="name parent *origin">
+    <joint name="${name}_joint" type="fixed">
+      <insert_block name="origin" />
+      <parent link="${parent}"/>
+      <child link="${name}_link" />
+    </joint>
+    <link name="${name}_link">
+      <visual>
+        <origin xyz="0 0 0" rpy="-1.57 3.14 0" />
+        <geometry>
+          <mesh filename="package://maxwell_defs/meshes/head_mount.stl" scale="1 1 1"/>
+        </geometry>
+        <material name="Black"/>
+      </visual>
+      <collision>
+        <origin xyz="0 0 0" rpy="0 0 0" />
+        <geometry>
+          <box size="0.0865 0.0047625 0.038"/>
+        </geometry>
+      </collision>
+    </link>
+  </macro>
   <!-- origin is center of head tilt rotation -->
   <macro name="maxwell_head" params="name parent *origin">
+    <joint name="${name}_joint" type="fixed">
+      <insert_block name="origin" />
+      <parent link="${parent}_link"/>
+      <child link="${name}_link"/>
+    </joint>
+    <link name="${name}_link"/>
+    <head_mount name="${name}_left_mount" parent="${name}_link">
+      <origin xyz="0 0.01905 0" rpy="0 0 0"/>
+    </head_mount>
+    <head_mount name="${name}_right_mount" parent="${name}_link">
+      <origin xyz="0 ${-0.01905-0.003175} 0" rpy="0 0 0"/>
+    </head_mount>
     <!-- Head pan -->
-    <dynamixel_ax12_pan parent="${parent}" name="${name}_pan_servo" color="Black">
-      <insert_block name="origin" />
+    <dynamixel_ax12_pan parent="${name}_link" name="${name}_pan_servo" color="Black">
+      <origin xyz="0.010 0 0.0254" rpy="0 0 0"/>
     </dynamixel_ax12_pan>
-    <ax12_side_revolute parent="${name}_pan_servo_link" name="${name}_pan" llimit="-2.617" ulimit="2.617" color="Orange">
+    <ax12_side_revolute parent="${name}_pan_servo_link" name="${name}_pan" llimit="-2.617" ulimit="2.617" vlimit="1.0" color="Orange">
       <origin xyz="0 0 ${AX12_WIDTH/2}" rpy="0 0 0"/>
     </ax12_side_revolute>
@@ -20,5 +55,5 @@
       <origin xyz="0 0 ${AX12_HEIGHT+0.003}" rpy="0 0 0"/>
     </dynamixel_ax12_tilt>
-    <ax12_hinge_revolute parent="${name}_tilt_servo_link" name="${name}_tilt" color="Orange">
+    <ax12_hinge_revolute parent="${name}_tilt_servo_link" name="${name}_tilt" llimit="-2.617" ulimit="2.617" vlimit="1.0" color="Orange">
      <origin xyz="0 0 0" rpy="0 0 0"/>
     </ax12_hinge_revolute>

File: maxwell/maxwell_defs/urdf/maxwell.urdf.xacro (robot description, xacro)
@@ -32,7 +32,7 @@
     <origin xyz="0 0 0" />
   </maxwell_gripper>
-  <!-- Kinect head -->
-  <maxwell_head name="head" parent="torso_link">
-    <origin xyz="0 0 ${column_height+0.0270375}"/>
+  <!-- Head -->
+  <maxwell_head name="head" parent="torso">
+    <origin xyz="0 0 ${column_height}"/>
   </maxwell_head>
 </robot>

Commit message: (maxwell_defs) update ax12 collision models

File: maxwell/maxwell_defs/urdf/arm.urdf.xacro (robot description, xacro)
@@ -123,7 +123,7 @@
       </visual>
       <collision>
-        <origin xyz="${0.0381/2} 0.0 -0.01241 " rpy="0 0 0" />
+        <origin xyz="${0.040/2} 0.0 ${-(0.0506-0.024)/2} " rpy="0 0 0" />
         <geometry>
-          <box size="0.0381 0.028 0.04762"/>
+          <box size="0.040 0.032 0.0501"/>
         </geometry>
       </collision>

File: maxwell/maxwell_defs/urdf/hardware/ax12.xacro (robot description, xacro)
@@ -25,7 +25,7 @@
       </visual>
       <collision>
-        <origin xyz="-0.01241 0.0 0.0" rpy="0 0 0" />
-        <geometry>
-          <box size="0.04762 0.028 0.038"/>
+        <origin xyz="${-0.0501/2+0.0116} 0.0 0.0" rpy="0 0 0" />
+        <geometry>
+          <box size="0.0501 0.032 0.040"/>
         </geometry>
       </collision>
@@ -54,7 +54,7 @@
       </visual>
       <collision>
-        <origin xyz="0.0 0.0 -0.01241" rpy="0 0 0" />
-        <geometry>
-          <box size="0.028 0.038 0.04762"/>
+        <origin xyz="0.0 0.0 ${-0.0501/2+0.0116}" rpy="0 0 0" />
+        <geometry>
+          <box size="0.032 0.040 0.0501"/>
         </geometry>
       </collision>

File: maxwell/maxwell_defs/urdf/head.urdf.xacro (robot description, xacro)
@@ -17,5 +17,5 @@
       </visual>
       <collision>
-        <origin xyz="0 0 0" rpy="0 0 0" />
+        <origin xyz="0 0 0" rpy="0 1.57 0" />
         <geometry>
           <box size="0.0865 0.0047625 0.038"/>

Commit message: (maxwell) rename max_lite to maxlite_defs, add elbow standoffs to maxwell

File: maxwell/maxwell_defs/urdf/arm.urdf.xacro (robot description, xacro)
@@ -2,5 +2,5 @@
 <robot>
   <!-- standoffs -->
-  <macro name="standoffs" params="name parent *origin">
+  <macro name="standoffs" params="name parent length *origin">
     <joint name="${name}_joint" type="fixed">
       <insert_block name="origin" />
@@ -10,14 +10,14 @@
     <link name="${name}_link">
       <visual>
-        <origin xyz="${0.0381/2} 0 0" rpy="0 0 0" />
+        <origin xyz="${length/2} 0 0" rpy="0 0 0" />
         <geometry>
-          <box size="0.0381 0.037 0.030"/>
+          <box size="${length} 0.037 0.030"/>
         </geometry>
         <material name="Black"/>
       </visual>
       <collision>
-        <origin xyz="${0.0381/2} 0 0" rpy="0 0 0" />
+        <origin xyz="${length/2} 0 0" rpy="0 0 0" />
         <geometry>
-          <box size="0.0381 0.037 0.030"/>
+          <box size="${length} 0.037 0.030"/>
         </geometry>
       </collision>
@@ -76,5 +76,5 @@
       <origin xyz="0 0 0.0" rpy="0 0 0"/>
     </rx64_hinge_hxl>
-    <standoffs parent="${name}_shoulder_lift_link" name="${name}_shoulder_standoff">
+    <standoffs parent="${name}_shoulder_lift_link" name="${name}_shoulder_standoff" length="0.0381">
       <origin xyz="${0.048+0.0235} 0 0.0" rpy="0 0 0"/>
     </standoffs>
@@ -89,4 +89,7 @@
       <origin xyz="0 0 0.0" rpy="0 0 0"/>
     </rx64_hinge_hxl>
+    <standoffs parent="${name}_elbow_flex_link" name="${name}_elbow_standoff" length="0">
+      <origin xyz="${0.048+0.0235} 0 0.0" rpy="0 0 0"/>
+    </standoffs>
     <!-- Wrist flex -->
     <rx64_side_fixed parent="${name}_elbow_flex_link" name="${name}_wrist_flex_fixed" color="Grey">

Commit message: (maxwell_defs) fix standoff link

File: maxwell/maxwell_defs/urdf/arm.urdf.xacro (robot description, xacro)
@@ -14,5 +14,5 @@
           <box size="${length} 0.037 0.030"/>
         </geometry>
-        <material name="Black"/>
+        <material name="Grey"/>
       </visual>
       <collision>
@@ -93,6 +93,6 @@
     </standoffs>
     <!-- Wrist flex -->
-    <rx64_side_fixed parent="${name}_elbow_flex_link" name="${name}_wrist_flex_fixed" color="Grey">
-      <origin xyz="${0.048+0.0235} 0 0" rpy="0 0 0"/>
+    <rx64_side_fixed parent="${name}_elbow_standoff_link" name="${name}_wrist_flex_fixed" color="Grey">
+      <origin xyz="0 0 0" rpy="0 0 0"/>
     </rx64_side_fixed>
     <dynamixel_rx64_tilt parent="${name}_wrist_flex_fixed_link" name="${name}_wrist_flex_servo" color="Black">

Commit message: (maxwell_defs) change 0 position of lift servo

File: maxwell/maxwell_defs/urdf/arm.urdf.xacro (robot description, xacro)
@@ -67,12 +67,12 @@
     </dynamixel_rx64_pan>
     <rx64_side_revolute parent="${name}_shoulder_pan_servo_link" name="${name}_shoulder_pan" llimit="-1.57" ulimit="1.57" vlimit="0.524" color="Grey">
-      <origin xyz="0 0 0.0235" rpy="0 -1.57 0"/>
+      <origin xyz="0 0 0.0235" rpy="0 0 0"/>
     </rx64_side_revolute>
     <!-- Shoulder lift -->
     <dynamixel_rx64_tilt parent="${name}_shoulder_pan_link" name="${name}_shoulder_lift_servo" color="Black">
-      <origin xyz="${0.0611-0.013+0.0045} 0 0" rpy="0 0 0"/>
+      <origin xyz="0 0 ${0.0611-0.013+0.0045}" rpy="0 -1.57 0"/>
     </dynamixel_rx64_tilt>
-    <rx64_hinge_hxl parent="${name}_shoulder_lift_servo_link" name="${name}_shoulder_lift" llimit="-0.2" ulimit="2.617" vlimit="0.524" color="Grey">
-      <origin xyz="0 0 0.0" rpy="0 0 0"/>
+    <rx64_hinge_hxl parent="${name}_shoulder_lift_servo_link" name="${name}_shoulder_lift" llimit="-1.77" ulimit="1.317" vlimit="0.524" color="Grey">
+      <origin xyz="0 0 0.0" rpy="0 1.57 0"/>
     </rx64_hinge_hxl>
     <standoffs parent="${name}_shoulder_lift_link" name="${name}_shoulder_standoff" length="0.0381">

File: maxwell/maxwell_defs/urdf/hardware/rx64.xacro (robot description, xacro)
@@ -62,5 +62,5 @@
     <joint name="${name}_joint" type="revolute">
       <insert_block name="origin" />
-       <axis xyz="1 0 0"/>
+       <axis xyz="0 0 1"/>
       <limit effort="30" velocity="${vlimit}" lower="${llimit}" upper="${ulimit}" />
       <parent link="${parent}"/>
@@ -76,5 +76,5 @@
       </inertial>
       <visual>
-        <origin xyz=" 0 0 0 " rpy="1.57 1.57 0" />
+        <origin xyz=" 0 0 0 " rpy="1.57 0 0" />
         <geometry>
           <mesh filename="package://maxwell_defs/meshes/rx64-side-bracket.stl" scale="1 1 1"/>
