Commit message: (maxwell_defs) update to Asus Xtion, add linear actuator visualization

File: maxwell/maxwell_defs/urdf/arm.urdf.xacro (robot description, xacro)
@@ -35,5 +35,5 @@
         <origin xyz="0 0 0" rpy="1.57 3.14 0" />
         <geometry>
-          <mesh filename="package://maxwell_defs/meshes/arm_mount.stl" scale="1 1 1"/>
+          <mesh filename="package://maxwell_defs/meshes/arm_mount.stl" scale="0.001 0.001 0.001"/>
         </geometry>
         <material name="Black"/>
@@ -52,13 +52,13 @@
     <joint name="${name}_base_joint" type="fixed">
       <insert_block name="origin" />
-      <parent link="${parent}_link"/>
+      <parent link="${parent}"/>
       <child link="${name}_link"/>
     </joint>
     <link name="${name}_link"/>
     <arm_mount name="${name}_left_mount" parent="${name}_link">
-      <origin xyz="-0.0611 0.0254 0" rpy="0 0 0"/>
+      <origin xyz="-0.0611 0.0254 -0.034" rpy="0 0 0"/>
     </arm_mount>
     <arm_mount name="${name}_right_mount" parent="${name}_link">
-      <origin xyz="-0.0611 ${-0.0254+0.0047625} 0" rpy="0 0 0"/>
+      <origin xyz="-0.0611 ${-0.0254} 0.034" rpy="3.14 0 0"/>
     </arm_mount>
     <!-- Shoulder pan -->

File: maxwell/maxwell_defs/urdf/head.urdf.xacro (robot description, xacro)
@@ -28,5 +28,5 @@
     <joint name="${name}_joint" type="fixed">
       <insert_block name="origin" />
-      <parent link="${parent}_link"/>
+      <parent link="${parent}"/>
       <child link="${name}_link"/>
     </joint>
@@ -58,32 +58,4 @@
      <origin xyz="0 0 0" rpy="0 0 0"/>
     </ax12_hinge_revolute>
-    <!-- Head sensor frame -->
-    <joint name="${name}_sensor_frame_joint" type="fixed">
-      <origin xyz="0 0 0.0425"/>
-      <parent link="${name}_tilt_link"/>
-      <child link="${name}_sensor_frame"/>
-    </joint>
-    <link name="${name}_sensor_frame">
-      <!--<visual>
-        <origin xyz="-0.03 0 0" rpy="0 0 -1.57" />
-        <geometry>
-          <mesh filename="package://maxwell_defs/meshes/kinect.stl" />
-        </geometry>
-        <material name="Black" />
-      </visual>
-      <collision>
-        <origin xyz="0 0 0" rpy="0 0 0" />
-        <geometry>
-          <box size="0.064 0.28 0.04"/>
-        </geometry>
-      </collision>-->
-    </link>
-    <!-- Openni Link
-    <joint name="openni_camera_joint" type="fixed">
-      <origin xyz="${calib_cam_x} ${calib_cam_y} ${calib_cam_z}" rpy="${calib_cam_rr} ${calib_cam_rp} ${calib_cam_ry}" />
-      <parent link="${name}_sensor_frame"/>
-      <child link="openni_camera"/>
-    </joint>
-    <link name="openni_camera"/>-->
   </macro>
 </robot>

File: maxwell/maxwell_defs/urdf/maxwell.urdf.xacro (robot description, xacro)
@@ -11,5 +11,5 @@
   <include filename="$(find maxwell_defs)/urdf/hardware/ax12.xacro" />
   <include filename="$(find maxwell_defs)/urdf/hardware/rx64.xacro" />
-  <include filename="$(find maxwell_defs)/urdf/sensors/kinect_camera.urdf.xacro" />
+  <include filename="$(find maxwell_defs)/urdf/sensors/xtion_camera.xacro" />
   <!-- The following included files set up definitions of parts of the robot body -->
   <include filename="$(find maxwell_defs)/urdf/base.urdf.xacro" />
@@ -22,5 +22,5 @@
   <armadillo_base name="base" color="Orange"/>
   <!-- Add Torso Upright -->
-  <maxwell_torso name="torso" parent="base">
+  <maxwell_torso name="torso" parent="base_link">
     <origin xyz="-0.00635 0 ${base_size_z+arm_height}" rpy="0 0 0"/>
   </maxwell_torso>
@@ -35,5 +35,5 @@
   <link name="arm_lift_link"/>
   <!-- Arm -->
-  <maxwell_arm name="arm" parent="arm_lift">
+  <maxwell_arm name="arm" parent="arm_lift_link">
     <origin xyz="0.0611 0 0" rpy="0 0 0"/>
   </maxwell_arm>
@@ -43,9 +43,9 @@
   </maxwell_gripper>
   <!-- Head -->
-  <maxwell_head name="head" parent="torso" color="Orange">
+  <maxwell_head name="head" parent="torso_link" color="Orange">
     <origin xyz="0 0 ${column_height-arm_height}" rpy="0 0 0"/>
   </maxwell_head>
-  <kinect_camera name="head_kinect" parent="head_sensor_frame">
-    <origin xyz="0 .07 .02" rpy="0 -.06 0"/> <!-- TODO: these values work, update underlying aspects for ASUS Xtion -->
-  </kinect_camera>
+  <xtion_camera name="head_camera" parent="head_tilt_link">
+    <origin xyz="0 0 0.026" rpy="0 0 0"/>
+  </xtion_camera>
 </robot>

File: maxwell/maxwell_defs/urdf/sensors/xtion_camera.xacro (robot description, xacro)
@@ -1,5 +1,5 @@
 <?xml version="1.0"?>
 <robot>
-  <macro name="kinect_camera" params="name parent *origin">
+  <macro name="xtion_camera" params="name parent *origin">
     <joint name="${name}_frame_joint" type="fixed">
       <insert_block name="origin" />
@@ -9,20 +9,20 @@
     <link name="${name}_frame">
       <visual>
-        <origin xyz="-0.03 -0.07 0" rpy="0 0 -1.57" />
+        <origin xyz="0 0 0" rpy="0 0 -1.57" />
         <geometry>
-          <mesh filename="package://maxwell_defs/meshes/kinect.stl" />
+          <mesh filename="package://maxwell_defs/meshes/xtion.stl" scale="0.001 0.001 0.001"/>
         </geometry>
         <material name="Black" />
       </visual>
       <collision>
-        <origin xyz="0 0 0" rpy="0 0 0" />
+        <origin xyz="0 0 0.032075" rpy="0 0 0" />
         <geometry>
-          <box size="0.064 0.28 0.04"/>
+          <box size="0.0381 0.1793875 0.0254"/>
         </geometry>
       </collision>
     </link>
-    <!-- kinect ir sensor physical attachment -->
+    <!-- ir sensor physical attachment -->
     <joint name="${name}_ir_joint" type="fixed">
-      <origin xyz="0 0 0" rpy="0 0 0"/>
+      <origin xyz="0.01905 -0.0269875 0.032075" rpy="0 0 0"/>
       <parent link="${name}_frame"/>
       <child link="${name}_ir_link"/>
@@ -36,5 +36,5 @@
       </visual>
     </link>
-    <!-- kinect ir sensor frame -->
+    <!-- ir sensor frame -->
     <joint name="${name}_ir_optical_frame_joint" type="fixed">
       <origin xyz="0 0 0" rpy="-1.57 0.0 -1.57" />
@@ -43,7 +43,7 @@
     </joint>
     <link name="${name}_ir_optical_frame"/>
-    <!-- kinect rgb sensor physical attachment -->
+    <!-- rgb sensor physical attachment -->
     <joint name="${name}_rgb_joint" type="fixed">
-      <origin xyz="0 -0.03 0" rpy="0 0 0"/>
+      <origin xyz="0 0.0777875 0" rpy="0 0 0"/>
       <parent link="${name}_ir_link"/>
       <child link="${name}_rgb_link"/>
@@ -57,5 +57,5 @@
       </visual>
     </link>
-    <!-- kinect rgb sensor frame -->
+    <!-- rgb sensor frame -->
     <joint name="${name}_rgb_optical_frame_joint" type="fixed">
       <origin xyz="0 0 0" rpy="-1.57 0.0 -1.57" />

File: maxwell/maxwell_defs/urdf/torso.urdf.xacro (robot description, xacro)
@@ -3,7 +3,6 @@
   <macro name="maxwell_torso" params="name parent *origin">
     <joint name="${name}_joint" type="fixed">
-      <axis xyz="0 1 0" />
       <insert_block name="origin" />
-      <parent link="${parent}_link"/>
+      <parent link="${parent}"/>
       <child link="${name}_link"/>
     </joint>
@@ -23,4 +22,24 @@
       </collision>
     </link>
+    <joint name="${name}_actuator_joint" type="fixed">
+      <origin xyz="0 0 0" rpy="0 0 0"/>
+      <parent link="${name}_link"/>
+      <child link="${name}_actuator_link"/>
+    </joint>
+    <link name="${name}_actuator_link">
+      <visual>
+        <origin xyz="-0.05 -0.0127 -0.560" rpy="0 0 3.14" />
+        <geometry>
+          <mesh filename="package://maxwell_defs/meshes/FA-35-TR.stl" scale="0.001 0.001 0.001"/>
+        </geometry>
+        <material name="Grey"/>
+      </visual>
+      <!--<collision>
+        <origin xyz="0 0 ${column_height/2 - arm_height}" rpy="0 0 0 " />
+        <geometry>
+          <box size="0.0254 0.0254 ${column_height}"/>
+        </geometry>
+      </collision>-->
+    </link>
   </macro>
 </robot>

Commit message: (maxwell_defs) update torso speed, add collision models for rotated brackets and arm mounts and torso actuator, remove elbow_standoffs

File: maxwell/maxwell_defs/urdf/arm.urdf.xacro (robot description, xacro)
@@ -33,5 +33,5 @@
     <link name="${name}_link">
       <visual>
-        <origin xyz="0 0 0" rpy="1.57 3.14 0" />
+        <origin xyz="0 0 -0.034" rpy="1.57 3.14 0" />
         <geometry>
           <mesh filename="package://maxwell_defs/meshes/arm_mount.stl" scale="0.001 0.001 0.001"/>
@@ -57,8 +57,8 @@
     <link name="${name}_link"/>
     <arm_mount name="${name}_left_mount" parent="${name}_link">
-      <origin xyz="-0.0611 0.0254 -0.034" rpy="0 0 0"/>
+      <origin xyz="-0.0611 0.0254 0" rpy="0 0 0"/>
     </arm_mount>
     <arm_mount name="${name}_right_mount" parent="${name}_link">
-      <origin xyz="-0.0611 ${-0.0254} 0.034" rpy="3.14 0 0"/>
+      <origin xyz="-0.0611 ${-0.0254} 0" rpy="3.14 0 0"/>
     </arm_mount>
     <!-- Shoulder pan -->
@@ -89,10 +89,10 @@
       <origin xyz="0 0 0.0" rpy="0 0 0"/>
     </rx64_hinge_hxl>
-    <standoffs parent="${name}_elbow_flex_link" name="${name}_elbow_standoff" length="0">
+   <!--<standoffs parent="${name}_elbow_flex_link" name="${name}_elbow_standoff" length="0">
       <origin xyz="${0.048+0.0235} 0 0.0" rpy="0 0 0"/>
-    </standoffs>
+    </standoffs>-->
     <!-- Wrist flex -->
-    <rx64_side_fixed parent="${name}_elbow_standoff_link" name="${name}_wrist_flex_fixed" color="Grey">
-      <origin xyz="0 0 0" rpy="0 0 0"/>
+    <rx64_side_fixed parent="${name}_elbow_flex_link" name="${name}_wrist_flex_fixed" color="Grey">
+      <origin xyz="${0.048+0.0235} 0 0" rpy="0 0 0"/>
     </rx64_side_fixed>
     <dynamixel_rx64_tilt parent="${name}_wrist_flex_fixed_link" name="${name}_wrist_flex_servo" color="Black">

File: maxwell/maxwell_defs/urdf/hardware/rx64.xacro (robot description, xacro)
@@ -83,7 +83,7 @@
       </visual>
       <collision>
-        <origin xyz="0.005 0 0.005" rpy="0 0 0" />
+        <origin xyz="0.000 0 0.005" rpy="0 0 0" />
         <geometry>
-          <box size="0.010 0.037 0.037"/>
+          <box size="0.037 0.037 0.010"/>
         </geometry>
       </collision>
@@ -112,5 +112,5 @@
       </visual>
       <collision>
-        <origin xyz="0.005 0 0.005" rpy="0 0 0" />
+        <origin xyz="0.005 0 0" rpy="0 0 0" />
         <geometry>
           <box size="0.010 0.037 0.037"/>

File: maxwell/maxwell_defs/urdf/maxwell.urdf.xacro (robot description, xacro)
@@ -28,5 +28,5 @@
   <joint name="arm_lift_joint" type="prismatic">
     <axis xyz="0 0 1" />
-    <limit lower="-0.464" upper="0" effort="30" velocity="0.013"/>
+    <limit lower="-0.464" upper="0" effort="30" velocity="0.0508"/>
     <origin xyz="0 0 0" rpy="0 0 0" />
     <parent link="torso_link"/>

File: maxwell/maxwell_defs/urdf/torso.urdf.xacro (robot description, xacro)
@@ -35,10 +35,10 @@
         <material name="Grey"/>
       </visual>
-      <!--<collision>
-        <origin xyz="0 0 ${column_height/2 - arm_height}" rpy="0 0 0 " />
+      <collision>
+        <origin xyz="-0.03 0 ${-0.650/2+.08}" rpy="0 0 0 " />
         <geometry>
-          <box size="0.0254 0.0254 ${column_height}"/>
+          <box size="0.03 0.0254 0.650"/>
         </geometry>
-      </collision>-->
+      </collision>
     </link>
   </macro>

Commit message: (maxwell_defs) update meshes/urdf for new arm

File: maxwell/maxwell_defs/urdf/arm.urdf.xacro (robot description, xacro)
@@ -73,29 +73,94 @@
       <origin xyz="0 0 ${0.0611-0.013+0.0045}" rpy="0 -1.57 0"/>
     </dynamixel_rx64_tilt>
-    <rx64_hinge_hxl parent="${name}_shoulder_lift_servo_link" name="${name}_shoulder_lift" llimit="-1.77" ulimit="1.317" vlimit="0.524" color="Grey">
-      <origin xyz="0 0 0.0" rpy="0 1.57 0"/>
-    </rx64_hinge_hxl>
-    <standoffs parent="${name}_shoulder_lift_link" name="${name}_shoulder_standoff" length="0.0381">
-      <origin xyz="${0.048+0.0235} 0 0.0" rpy="0 0 0"/>
-    </standoffs>
+    <joint name="${name}_shoulder_lift_joint" type="revolute">
+      <origin xyz="0 0 0" rpy="0 1.57 0"/>
+      <axis xyz="0 1 0"/>
+      <limit effort="30" velocity="0.524" lower="-1.77" upper="1.317" />
+      <parent link="${name}_shoulder_lift_servo_link"/>
+      <child link="${name}_shoulder_lift_link" />
+    </joint>
+    <link name="${name}_shoulder_lift_link">
+      <inertial>
+        <mass value="0.00001" />
+        <origin xyz="0 0 0" />
+        <inertia ixx="1.0" ixy="0.0" ixz="0.0"
+          iyy="1.0" iyz="0.0"
+          izz="1.0" />
+      </inertial>
+      <visual>
+        <origin xyz="0 0 0" rpy="-1.57 0 0" />
+        <geometry>
+          <mesh filename="package://maxwell_defs/meshes/arm_mx64_upper.stl" scale="1 1 1"/>
+        </geometry>
+        <material name="Black"/>
+      </visual>
+      <collision>
+        <origin xyz="0.08 0.0 0.0" rpy="0 0 0" />
+        <geometry>
+          <box size="0.204 0.053 0.044"/>
+        </geometry>
+      </collision>
+    </link>
     <!-- Elbow -->
-    <rx64_side_fixed parent="${name}_shoulder_standoff_link" name="${name}_elbow_flex_fixed" color="Grey">
-      <origin xyz="0.0381 0 0" rpy="0 0 0"/>
-    </rx64_side_fixed>
-    <dynamixel_rx64_tilt parent="${name}_elbow_flex_fixed_link" name="${name}_elbow_flex_servo" color="Black">
-      <origin xyz="${0.0611-0.013+0.0045} 0 0" rpy="0 0 0"/>
-    </dynamixel_rx64_tilt>
-    <rx64_hinge_hxl parent="${name}_elbow_flex_servo_link" name="${name}_elbow_flex" llimit="-1.57" ulimit="2.617" vlimit="0.524" color="Grey">
-      <origin xyz="0 0 0.0" rpy="0 0 0"/>
-    </rx64_hinge_hxl>
-   <!--<standoffs parent="${name}_elbow_flex_link" name="${name}_elbow_standoff" length="0">
-      <origin xyz="${0.048+0.0235} 0 0.0" rpy="0 0 0"/>
-    </standoffs>-->
+    <joint name="${name}_elbow_flex_joint" type="revolute">
+      <origin xyz="0.16 0 0" rpy="0 0 0"/>
+      <axis xyz="0 1 0"/>
+      <limit effort="30" velocity="0.524" lower="-1.57" upper="2.617" />
+      <parent link="${name}_shoulder_lift_link"/>
+      <child link="${name}_elbow_flex_link" />
+    </joint>
+    <link name="${name}_elbow_flex_link">
+      <inertial>
+        <mass value="0.00001" />
+        <origin xyz="0 0 0" />
+        <inertia ixx="1.0" ixy="0.0" ixz="0.0"
+          iyy="1.0" iyz="0.0"
+          izz="1.0" />
+      </inertial>
+      <visual>
+        <origin xyz=" 0 0 0 " rpy="1.57 -1.57 0" />
+        <geometry>
+          <mesh filename="package://maxwell_defs/meshes/rx64.stl" scale="1 1 1"/>
+        </geometry>
+        <material name="Black"/>
+      </visual>
+      <collision>
+        <origin xyz="${(0.0611-0.026)/2} 0 0" rpy="0 0 0" />
+        <geometry>
+          <box size="0.0611 0.0470 0.0420"/>
+        </geometry>
+      </collision>
+    </link>
+    <!-- Forearm -->
+    <joint name="${name}_forearm_fixed_joint" type="fixed">
+      <origin xyz="0 0 0" rpy="0 0 0"/>
+      <parent link="${name}_elbow_flex_link"/>
+      <child link="${name}_forearm_link" />
+    </joint>
+    <link name="${name}_forearm_link">
+      <inertial>
+        <mass value="0.00001" />
+        <origin xyz="0 0 0" />
+        <inertia ixx="1.0" ixy="0.0" ixz="0.0"
+          iyy="1.0" iyz="0.0"
+          izz="1.0" />
+      </inertial>
+      <visual>
+        <origin xyz="0 0 0" rpy="-1.57 0 0" />
+        <geometry>
+          <mesh filename="package://maxwell_defs/meshes/arm_mx64_forearm.stl" scale="1 1 1"/>
+        </geometry>
+        <material name="Black"/>
+      </visual>
+      <collision>
+        <origin xyz="0.0625 0.0 0.0" rpy="0 0 0" />
+        <geometry>
+          <box size="0.03 0.053 0.044"/>
+        </geometry>
+      </collision>
+    </link>
     <!-- Wrist flex -->
-    <rx64_side_fixed parent="${name}_elbow_flex_link" name="${name}_wrist_flex_fixed" color="Grey">
-      <origin xyz="${0.048+0.0235} 0 0" rpy="0 0 0"/>
-    </rx64_side_fixed>
-    <dynamixel_rx64_tilt parent="${name}_wrist_flex_fixed_link" name="${name}_wrist_flex_servo" color="Black">
-      <origin xyz="${0.0611-0.013+0.0045} 0 0" rpy="0 0 0"/>
+    <dynamixel_rx64_tilt parent="${name}_forearm_link" name="${name}_wrist_flex_servo" color="Black">
+      <origin xyz="0.125 0 0" rpy="0 0 0"/>
     </dynamixel_rx64_tilt>
     <rx64_hinge parent="${name}_wrist_flex_servo_link" name="${name}_wrist_flex" llimit="-1.57" ulimit="1.57" vlimit="0.785" color="Grey">

File: maxwell/maxwell_defs/urdf/hardware/rx64.xacro (robot description, xacro)
@@ -90,64 +90,4 @@
     </link>
   </macro>
-  <macro name="rx64_side_fixed" params="parent name color *origin">
-    <joint name="${name}_joint" type="fixed">
-      <insert_block name="origin" />
-      <parent link="${parent}"/>
-      <child link="${name}_link" />
-    </joint>
-    <link name="${name}_link">
-      <inertial>
-        <mass value="0.00001" />
-        <origin xyz="0 0 0" />
-        <inertia ixx="1.0" ixy="0.0" ixz="0.0"
-          iyy="1.0" iyz="0.0"
-          izz="1.0" />
-      </inertial>
-      <visual>
-        <origin xyz=" 0 0 0 " rpy="1.57 1.57 0" />
-        <geometry>
-          <mesh filename="package://maxwell_defs/meshes/rx64-side-bracket.stl" scale="1 1 1"/>
-        </geometry>
-        <material name="${color}"/>
-      </visual>
-      <collision>
-        <origin xyz="0.005 0 0" rpy="0 0 0" />
-        <geometry>
-          <box size="0.010 0.037 0.037"/>
-        </geometry>
-      </collision>
-    </link>
-  </macro>
-  <macro name="rx64_hinge_hxl" params="parent name color llimit ulimit vlimit *origin">
-    <joint name="${name}_joint" type="revolute">
-      <insert_block name="origin" />
-       <axis xyz="0 1 0"/>
-      <limit effort="30" velocity="${vlimit}" lower="${llimit}" upper="${ulimit}" />
-      <parent link="${parent}"/>
-      <child link="${name}_link" />
-    </joint>
-    <link name="${name}_link">
-      <inertial>
-        <mass value="0.00001" />
-        <origin xyz="0 0 0" />
-        <inertia ixx="1.0" ixy="0.0" ixz="0.0"
-          iyy="1.0" iyz="0.0"
-          izz="1.0" />
-      </inertial>
-      <visual>
-        <origin xyz="${0.048+0.0235} -0.0235 0.015" rpy="-1.57 0 1.57" />
-        <geometry>
-          <mesh filename="package://maxwell_defs/meshes/rx64-hxl.stl" scale="1 1 1"/>
-        </geometry>
-        <material name="${color}"/>
-      </visual>
-      <collision>
-        <origin xyz="${(0.048+0.0235)/2} 0.0 0.0" rpy="0 0 0" />
-        <geometry>
-          <box size="${0.048+0.0235} 0.056 0.031"/>
-        </geometry>
-      </collision>
-    </link>
-  </macro>
   <macro name="rx64_hinge" params="parent name color llimit ulimit vlimit *origin">
     <joint name="${name}_joint" type="revolute">
