Commit message: (maxwell_defs) update urdf

File: maxwell/maxwell_defs/urdf/maxwell.urdf.xacro (robot description, xacro)
@@ -1,30 +1,34 @@
 <?xml version="1.0"?>
 <robot name="maxwell" >
-  <!-- interactive calibration output:
-        [ INFO] [1310855144.314114846]: -0.0184416, -7.34934e-11, 0.07469, 0.0120684, 0.00708517, -8.5516e-05, 0.999902
-        [ INFO] [1310858627.105328692]: 0.00927514, 0.00208817, 0.0877625, 0.0240435, 0.0424938, 0.00594516, 0.998789
-        [ INFO] [1310858627.105465208]: 0.00927514, 0.00208817, 0.0877625, 0.048728, 0.0847001, 0.0139699
+  <!-- Calibration from 8/7
+  <property name='calib_cam_x' value='-0.000859868' />
+  <property name='calib_cam_y' value='0.0171667' />
+  <property name='calib_cam_z' value='0.0192186' />
+  <property name='calib_cam_rr' value='-0.0432624' />
+  <property name='calib_cam_rp' value='-0.0226177' />
+  <property name='calib_cam_ry' value='0.00714413' />
   -->
-  <!--<property name="calib_cam_x" value="0" />
+  <!-- Calibration from 8/8
+  <property name='calib_cam_x' value='-0.00515338' />
+  <property name='calib_cam_y' value='0.0131489' />
+  <property name='calib_cam_z' value='0.0169829' />
+  <property name='calib_cam_rr' value='-0.0397998' />
+  <property name='calib_cam_rp' value='-0.0241423' />
+  <property name='calib_cam_ry' value='0.00627637' />
+  -->
+  <property name='calib_cam_x' value='0.00468423' />
+  <property name='calib_cam_y' value='0.0060704' />
+  <property name='calib_cam_z' value='0.0118428' />
+  <property name='calib_cam_rr' value='-0.024976' />
+  <property name='calib_cam_rp' value='-0.0119664' />
+  <property name='calib_cam_ry' value='0.0228755' />
+  <!--
+  <property name="calib_cam_x" value="0" />
   <property name="calib_cam_y" value="0" />
   <property name="calib_cam_z" value="0" />
   <property name="calib_cam_rr" value="0" />
   <property name="calib_cam_rp" value="0" />
-  <property name="calib_cam_ry" value="0" />-->
-  <property name='calib_cam_x' value='-0.000859868' />
-  <property name='calib_cam_y' value='0.0171667' />
-  <!--<property name='calib_cam_y' value='0.0743167' />-->
-  <property name='calib_cam_z' value='0.0192186' />
-  <property name='calib_cam_rr' value='-0.0432624' />
-  <property name='calib_cam_rp' value='-0.0226177' />
-  <property name='calib_cam_ry' value='0.00714413' />
-  <!--<property name="calib_cam_x" value="0.00927514" />
-  <property name="calib_cam_y" value="-0.015" />
-  <property name="old_calib_cam_y" value="0.00208817" />
-  <property name="calib_cam_z" value="0.0877625" />
-  <property name="calib_cam_rr" value="0.048728" />
-  <property name="calib_cam_rp" value="0.0847001" />
-  <property name="calib_cam_ry" value="0.0359699" />
-  <property name="old_calib_cam_ry" value="0.0139699" />-->
+  <property name="calib_cam_ry" value="0" />
+  -->
   <property name="ax12_height" value="0.04762" />
   <property name="ax12_width" value="0.0381" />
@@ -32,5 +36,6 @@
   <property name="ax12_center" value="0.0385" />
   <!-- height properties -->
-  <property name="arm_height" value="0.885825" /> <!-- height to shoulder lift rotation -->
+  <!--<property name="arm_height" value="0.911225" />-->
+  <property name="arm_height" value="0.885825" /><!-- height to shoulder lift rotation -->
   <property name="column_height" value="1.397" /> <!-- height to neck tilt rotation -->
   <!-- The following included files set up definitions of parts of the robot body -->
@@ -57,5 +62,6 @@
   <!-- Kinect head -->
   <maxwell_head name="head" parent="base">
-    <origin xyz="0.0157 0 ${column_height}"/>
+    <!--<origin xyz="0.0157 0 ${column_height}"/>-->
+    <origin xyz="${0.0157+0.05715/2} -0.005 ${column_height}"/>
   </maxwell_head>
 </robot>

Commit message: (maxwell_defs) add RPY to many items in URDF, adjust heights of column/arm

File: maxwell/maxwell_defs/urdf/maxwell.urdf.xacro (robot description, xacro)
@@ -7,6 +7,6 @@
   <property name='calib_cam_rp' value='0.00482693' />
   <property name='calib_cam_ry' value='0.0643122' />
-  <property name="arm_height" value="0.6619375 " /> <!-- deck to arm_link -->
-  <property name="column_height" value="1.171575" /> <!-- deck to top of 80/20: 46-1/8" -->
+  <property name="arm_height" value="0.7239"/> <!-- deck to arm_link at max height-->
+  <property name="column_height" value="1.160075" /> <!-- deck to top of 80/20: 46-1/8" -->
   <include filename="$(find maxwell_defs)/urdf/hardware/ax12.xacro" />
   <include filename="$(find maxwell_defs)/urdf/hardware/rx64.xacro" />
@@ -23,20 +23,20 @@
   <!-- Add Torso Upright -->
   <maxwell_torso name="torso" parent="base">
-    <origin xyz="-0.00635 0 ${base_size_z}"/>
+    <origin xyz="-0.00635 0 ${base_size_z}" rpy="0 -0.01 0"/>
   </maxwell_torso>
   <!-- Arm -->
   <maxwell_arm name="arm" parent="torso">
-    <origin xyz="0.0611 0 ${arm_height}"/>
+    <origin xyz="0.0611 0 ${arm_height}" rpy="0 0 0"/>
   </maxwell_arm>
   <!-- Gripper -->
   <maxwell_gripper name="gripper" parent="arm_wrist_roll" color="Orange">
-    <origin xyz="0 0 0" />
+    <origin xyz="0 0 0" rpy="0 0 0" />
   </maxwell_gripper>
   <!-- Head -->
   <maxwell_head name="head" parent="torso" color="Orange">
-    <origin xyz="0 0 ${column_height}"/>
+    <origin xyz="0 0 ${column_height}" rpy="0 0 0"/>
   </maxwell_head>
   <kinect_camera name="head_kinect" parent="head_sensor_frame">
-    <origin xyz="0 0 0"/>
+    <origin xyz="0 .07 .02" rpy="0 -.06 0"/> <!-- TODO: these values work, update underlying aspects for ASUS Xtion -->
   </kinect_camera>
 </robot>

File: maxwell/maxwell_defs/urdf/sensors/kinect_camera.urdf.xacro (robot description, xacro)
@@ -9,5 +9,5 @@
     <link name="${name}_frame">
       <visual>
-        <origin xyz="-0.03 0 0" rpy="0 0 -1.57" />
+        <origin xyz="-0.03 -0.07 0" rpy="0 0 -1.57" />
         <geometry>
           <mesh filename="package://maxwell_defs/meshes/kinect.stl" />

Commit message: (maxwell_defs) move torso_link up to arm 0 position, add arm_lift_joint

File: maxwell/maxwell_defs/urdf/maxwell.urdf.xacro (robot description, xacro)
@@ -23,9 +23,18 @@
   <!-- Add Torso Upright -->
   <maxwell_torso name="torso" parent="base">
-    <origin xyz="-0.00635 0 ${base_size_z}" rpy="0 -0.01 0"/>
+    <origin xyz="-0.00635 0 ${base_size_z+arm_height}" rpy="0 0 0"/>
   </maxwell_torso>
+  <!-- Live joint between torso and arm -->
+  <joint name="arm_lift_joint" type="prismatic">
+    <axis xyz="0 0 1" />
+    <limit lower="-0.464" upper="0" effort="30" velocity="0.013"/>
+    <origin xyz="0 0 0" rpy="0 0 0" />
+    <parent link="torso_link"/>
+    <child link="arm_lift_link"/>
+  </joint>
+  <link name="arm_lift_link"/>
   <!-- Arm -->
-  <maxwell_arm name="arm" parent="torso">
-    <origin xyz="0.0611 0 ${arm_height}" rpy="0 0 0"/>
+  <maxwell_arm name="arm" parent="arm_lift">
+    <origin xyz="0.0611 0 0" rpy="0 0 0"/>
   </maxwell_arm>
   <!-- Gripper -->
@@ -35,5 +44,5 @@
   <!-- Head -->
   <maxwell_head name="head" parent="torso" color="Orange">
-    <origin xyz="0 0 ${column_height}" rpy="0 0 0"/>
+    <origin xyz="0 0 ${column_height-arm_height}" rpy="0 0 0"/>
   </maxwell_head>
   <kinect_camera name="head_kinect" parent="head_sensor_frame">

File: maxwell/maxwell_defs/urdf/torso.urdf.xacro (robot description, xacro)
@@ -10,5 +10,5 @@
     <link name="${name}_link">
       <visual>
-        <origin xyz="0 0 ${column_height/2}" rpy="0 0 0 " />
+        <origin xyz="0 0 ${column_height/2 - arm_height}" rpy="0 0 0 " />
         <geometry>
           <box size="0.0254 0.0254 ${column_height}"/>
@@ -17,5 +17,5 @@
       </visual>
       <collision>
-        <origin xyz="0 0 ${column_height/2}" rpy="0 0 0 " />
+        <origin xyz="0 0 ${column_height/2 - arm_height}" rpy="0 0 0 " />
         <geometry>
           <box size="0.0254 0.0254 ${column_height}"/>

Commit message: (maxwell_defs) add no_arm, update launch files

File: maxwell/maxwell_defs/urdf/maxwell.urdf.xacro (robot description, xacro)
@@ -1,11 +1,5 @@
 <?xml version="1.0"?>
 <robot name="maxwell" >
-  <property name='calib_cam_x' value='0.00259672' />
-  <property name='calib_cam_y' value='0.0307021' />
-  <property name='calib_cam_z' value='0.0133213' />
-  <property name='calib_cam_rr' value='-0.0829819' />
-  <property name='calib_cam_rp' value='0.00482693' />
-  <property name='calib_cam_ry' value='0.0643122' />
-  <property name="arm_height" value="0.7239"/> <!-- deck to arm_link at max height-->
+  <property name="arm_height" value="0.6731"/> <!-- deck to arm_link at max height-->
   <property name="column_height" value="1.160075" /> <!-- deck to top of 80/20: 46-1/8" -->
   <include filename="$(find maxwell_defs)/urdf/hardware/ax12.xacro" />

File: maxwell/maxwell_defs/urdf/sensors/kinect_camera.urdf.xacro (robot description, xacro)
@@ -9,5 +9,6 @@
     <link name="${name}_frame">
       <visual>
-        <origin xyz="-0.03 -0.07 0" rpy="0 0 -1.57" />
+        <origin xyz="-0.03 0 0.02" rpy="0 0 -1.57" />
+        <!--origin xyz="-0.03 -0.07 0" rpy="0 0 -1.57"-->
         <geometry>
           <mesh filename="package://maxwell_defs/meshes/kinect.stl" />

Commit message: (maxwell_defs) update urdf with some tweaks to better jumpstart calibration

File: maxwell/maxwell_defs/urdf/maxwell.urdf.xacro (robot description, xacro)
@@ -1,6 +1,6 @@
 <?xml version="1.0"?>
 <robot name="maxwell" >
-  <property name="arm_height" value="0.6731"/> <!-- deck to arm_link at max height-->
-  <property name="column_height" value="1.160075" /> <!-- deck to top of 80/20: 46-1/8" -->
+  <property name="arm_height" value="0.6604"/> <!-- deck to arm_link at max height-->
+  <property name="column_height" value="1.172775" /> <!-- deck to top of 80/20 -->
   <include filename="$(find maxwell_defs)/urdf/hardware/ax12.xacro" />
   <include filename="$(find maxwell_defs)/urdf/hardware/rx64.xacro" />

File: maxwell/maxwell_defs/urdf/sensors/xtion_camera.xacro (robot description, xacro)
@@ -45,5 +45,5 @@
     <!-- rgb sensor physical attachment -->
     <joint name="${name}_rgb_joint" type="fixed">
-      <origin xyz="0 0.0777875 0" rpy="0 0 0"/>
+      <origin xyz="0 0.0552875 0" rpy="0 -0.08 0"/>
       <parent link="${name}_ir_link"/>
       <child link="${name}_rgb_link"/>
